File: JTAG.sch (KiCad schematic (older format))
At the start: 1 part, among them J2 JTAG

Commit message: Before I remove ESP32
Changed lines of the file:
@@
 $Descr A4 11693 8268
 encoding utf-8
-Sheet 9 10
+Sheet 7 11
 Title ""
 Date ""
@@
 U 1 1 61B2217D
 P 4450 3650
+AR Path="/61B15767/61B2217D" Ref="J2"  Part="1"
+AR Path="/61AA52C4/61B2217D" Ref="J?"  Part="1"
 F 0 "J2" H 4500 4050 50  0000 C CNN
 F 1 "JTAG" H 4500 3250 50  0000 C CNN
@@
 U 1 1 61B22961
 P 4250 3950
+AR Path="/61B15767/61B22961" Ref="#PWR0127"  Part="1"
+AR Path="/61AA52C4/61B22961" Ref="#PWR?"  Part="1"
 F 0 "#PWR0127" H 4250 3700 50  0001 C CNN
-F 1 "GND" H 4255 3777 50  0000 C CNN
+F 1 "GND" H 4250 3800 50  0000 C CNN
 F 2 "" H 4250 3950 50  0001 C CNN
 F 3 "" H 4250 3950 50  0001 C CNN
@@
 U 1 1 61B2334F
 P 4750 3350
+AR Path="/61B15767/61B2334F" Ref="#PWR0128"  Part="1"
+AR Path="/61AA52C4/61B2334F" Ref="#PWR?"  Part="1"
 F 0 "#PWR0128" H 4750 3200 50  0001 C CNN
 F 1 "+3V3" H 4750 3500 50  0000 C CNN
