File: Buf.sch (KiCad schematic (older format))
At the start: 24 parts, among them U13 74AHCT573, U15 74AHCT573, U16 74AHCT573, U17 74AHCT573, U18 74AHCT573, U19 74AHCT573, U2 74AHCT573, U20 74AHCT573, U21 74AHCT573, U22 74AHCT573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

Commit message: Moving toward new update system
Parts:
- C33, C34, C35, C36, C37, C38, C39, C40, C41, C42, C43, C44: LCSC Part (none) -> C23630
- U13, U15, U16, U17, U18, U19, U2, U20, U21, U22, U23, U24: value 74AHCT573 -> 74AHCT573PW; LCSC Part (none) -> C141311
Changed lines of the file:
@@
 P 2400 4650
 F 0 "U15" H 2400 5250 50  0000 C CNN
-F 1 "74AHCT573" V 2400 4650 50  0000 C CNN
+F 1 "74AHCT573PW" V 2400 4650 50  0000 C CNN
 F 2 "stdpads:TSSOP-20_4.4x6.5mm_P0.65mm" H 2400 4000 50  0001 C TNN
 F 3 "" H 2400 4750 60  0001 C CNN
+F 4 "C141311" H 2400 4650 50  0001 C CNN "LCSC Part"
 	1    2400 4650
 	-1   0    0    -1
@@
 F 2 "stdpads:C_0603" H 2300 7300 50  0001 C CNN
 F 3 "~" H 2300 7300 50  0001 C CNN
+F 4 "C23630" H 2300 7300 50  0001 C CNN "LCSC Part"
 	1    2300 7300
 	1    0    0    -1
@@
 F 2 "stdpads:C_0603" H 2700 7300 50  0001 C CNN
 F 3 "~" H 2700 7300 50  0001 C CNN
+F 4 "C23630" H 2700 7300 50  0001 C CNN "LCSC Part"
 	1    2700 7300
 	1    0    0    -1
@@
 F 2 "stdpads:C_0603" H 3100 7300 50  0001 C CNN
 F 3 "~" H 3100 7300 50  0001 C CNN
+F 4 "C23630" H 3100 7300 50  0001 C CNN "LCSC Part"
 	1    3100 7300
 	1    0    0    -1
@@
 F 2 "stdpads:C_0603" H 1900 7300 50  0001 C CNN
 F 3 "~" H 1900 7300 50  0001 C CNN
+F 4 "C23630" H 1900 7300 50  0001 C CNN "LCSC Part"
 	1    1900 7300
 	1    0    0    -1
@@
 F 2 "stdpads:C_0603" H 3900 7300 50  0001 C CNN
 F 3 "~" H 3900 7300 50  0001 C CNN
+F 4 "C23630" H 3900 7300 50  0001 C CNN "LCSC Part"
 	1    3900 7300
 	1    0    0    -1
@@
 F 2 "stdpads:C_0603" H 3500 7300 50  0001 C CNN
 F 3 "~" H 3500 7300 50  0001 C CNN
+F 4 "C23630" H 3500 7300 50  0001 C CNN "LCSC Part"
 	1    3500 7300
 	1    0    0    -1
@@
 F 2 "stdpads:C_0603" H 2300 6900 50  0001 C CNN
 F 3 "~" H 2300 6900 50  0001 C CNN
+F 4 "C23630" H 2300 6900 50  0001 C CNN "LCSC Part"
 	1    2300 6900
 	1    0    0    -1
@@
 F 2 "stdpads:C_0603" H 2700 6900 50  0001 C CNN
 F 3 "~" H 2700 6900 50  0001 C CNN
+F 4 "C23630" H 2700 6900 50  0001 C CNN "LCSC Part"
 	1    2700 6900
 	1    0    0    -1
@@
 F 2 "stdpads:C_0603" H 3100 6900 50  0001 C CNN
 F 3 "~" H 3100 6900 50  0001 C CNN
+F 4 "C23630" H 3100 6900 50  0001 C CNN "LCSC Part"
 	1    3100 6900
 	1    0    0    -1
@@
 F 2 "stdpads:C_0603" H 1900 6900 50  0001 C CNN
 F 3 "~" H 1900 6900 50  0001 C CNN
+F 4 "C23630" H 1900 6900 50  0001 C CNN "LCSC Part"
 	1    1900 6900
 	1    0    0    -1
@@
 F 2 "stdpads:C_0603" H 3900 6900 50  0001 C CNN
 F 3 "~" H 3900 6900 50  0001 C CNN
+F 4 "C23630" H 3900 6900 50  0001 C CNN "LCSC Part"
 	1    3900 6900
 	1    0    0    -1
@@
 F 2 "stdpads:C_0603" H 3500 6900 50  0001 C CNN
 F 3 "~" H 3500 6900 50  0001 C CNN
+F 4 "C23630" H 3500 6900 50  0001 C CNN "LCSC Part"
 	1    3500 6900
 	1    0    0    -1
@@
 P 3700 4650
 F 0 "U18" H 3700 5250 50  0000 C CNN
-F 1 "74AHCT573" V 3700 4650 50  0000 C CNN
+F 1 "74AHCT573PW" V 3700 4650 50  0000 C CNN
 F 2 "stdpads:TSSOP-20_4.4x6.5mm_P0.65mm" H 3700 4000 50  0001 C TNN
 F 3 "" H 3700 4750 60  0001 C CNN
+F 4 "C141311" H 3700 4650 50  0001 C CNN "LCSC Part"
 	1    3700 4650
 	-1   0    0    -1
@@
 P 2400 5850
 F 0 "U13" H 2400 6450 50  0000 C CNN
-F 1 "74AHCT573" V 2400 5850 50  0000 C CNN
+F 1 "74AHCT573PW" V 2400 5850 50  0000 C CNN
 F 2 "stdpads:TSSOP-20_4.4x6.5mm_P0.65mm" H 2400 5200 50  0001 C TNN
 F 3 "" H 2400 5950 60  0001 C CNN
+F 4 "C141311" H 2400 5850 50  0001 C CNN "LCSC Part"
 	1    2400 5850
 	-1   0    0    -1
@@
 P 3700 5850
 F 0 "U17" H 3700 6450 50  0000 C CNN
-F 1 "74AHCT573" V 3700 5850 50  0000 C CNN
+F 1 "74AHCT573PW" V 3700 5850 50  0000 C CNN
 F 2 "stdpads:TSSOP-20_4.4x6.5mm_P0.65mm" H 3700 5200 50  0001 C TNN
 F 3 "" H 3700 5950 60  0001 C CNN
+F 4 "C141311" H 3700 5850 50  0001 C CNN "LCSC Part"
 	1    3700 5850
 	-1   0    0    -1
@@
 P 3700 3450
 F 0 "U2" H 3700 4050 50  0000 C CNN
-F 1 "74AHCT573" V 3700 3450 50  0000 C CNN
+F 1 "74AHCT573PW" V 3700 3450 50  0000 C CNN
 F 2 "stdpads:TSSOP-20_4.4x6.5mm_P0.65mm" H 3700 2800 50  0001 C TNN
 F 3 "" H 3700 3550 60  0001 C CNN
+F 4 "C141311" H 3700 3450 50  0001 C CNN "LCSC Part"
 	1    3700 3450
 	-1   0    0    -1
@@
 P 2400 3450
 F 0 "U16" H 2400 4050 50  0000 C CNN
-F 1 "74AHCT573" V 2400 3450 50  0000 C CNN
+F 1 "74AHCT573PW" V 2400 3450 50  0000 C CNN
 F 2 "stdpads:TSSOP-20_4.4x6.5mm_P0.65mm" H 2400 2800 50  0001 C TNN
 F 3 "" H 2400 3550 60  0001 C CNN
+F 4 "C141311" H 2400 3450 50  0001 C CNN "LCSC Part"
 	1    2400 3450
 	-1   0    0    -1
@@
 P 8000 5550
 F 0 "U22" H 8000 6150 50  0000 C CNN
-F 1 "74AHCT573" V 8000 5550 50  0000 C CNN
+F 1 "74AHCT573PW" V 8000 5550 50  0000 C CNN
 F 2 "stdpads:TSSOP-20_4.4x6.5mm_P0.65mm" H 8000 4900 50  0001 C TNN
 F 3 "" H 8000 5650 60  0001 C CNN
+F 4 "C141311" H 8000 5550 50  0001 C CNN "LCSC Part"
 	1    8000 5550
 	1    0    0    -1
@@
 P 8000 1650
 F 0 "U19" H 8000 2250 50  0000 C CNN
-F 1 "74AHCT573" V 8000 1650 50  0000 C CNN
+F 1 "74AHCT573PW" V 8000 1650 50  0000 C CNN
 F 2 "stdpads:TSSOP-20_4.4x6.5mm_P0.65mm" H 8000 1000 50  0001 C TNN
 F 3 "" H 8000 1750 60  0001 C CNN
+F 4 "C141311" H 8000 1650 50  0001 C CNN "LCSC Part"
 	1    8000 1650
 	-1   0    0    -1
@@
 P 9300 1650
 F 0 "U23" H 9300 2250 50  0000 C CNN
-F 1 "74AHCT573" V 9300 1650 50  0000 C CNN
+F 1 "74AHCT573PW" V 9300 1650 50  0000 C CNN
 F 2 "stdpads:TSSOP-20_4.4x6.5mm_P0.65mm" H 9300 1000 50  0001 C TNN
 F 3 "" H 9300 1750 60  0001 C CNN
+F 4 "C141311" H 9300 1650 50  0001 C CNN "LCSC Part"
 	1    9300 1650
 	-1   0    0    -1
@@
 P 8000 2950
 F 0 "U20" H 8000 3550 50  0000 C CNN
-F 1 "74AHCT573" V 8000 2950 50  0000 C CNN
+F 1 "74AHCT573PW" V 8000 2950 50  0000 C CNN
 F 2 "stdpads:TSSOP-20_4.4x6.5mm_P0.65mm" H 8000 2300 50  0001 C TNN
 F 3 "" H 8000 3050 60  0001 C CNN
+F 4 "C141311" H 8000 2950 50  0001 C CNN "LCSC Part"
 	1    8000 2950
 	1    0    0    -1
@@
 P 8000 4250
 F 0 "U21" H 8000 4850 50  0000 C CNN
-F 1 "74AHCT573" V 8000 4250 50  0000 C CNN
+F 1 "74AHCT573PW" V 8000 4250 50  0000 C CNN
 F 2 "stdpads:TSSOP-20_4.4x6.5mm_P0.65mm" H 8000 3600 50  0001 C TNN
 F 3 "" H 8000 4350 60  0001 C CNN
+F 4 "C141311" H 8000 4250 50  0001 C CNN "LCSC Part"
 	1    8000 4250
 	-1   0    0    -1
@@
 P 9300 4250
 F 0 "U24" H 9300 4850 50  0000 C CNN
-F 1 "74AHCT573" V 9300 4250 50  0000 C CNN
+F 1 "74AHCT573PW" V 9300 4250 50  0000 C CNN
 F 2 "stdpads:TSSOP-20_4.4x6.5mm_P0.65mm" H 9300 3600 50  0001 C TNN
 F 3 "" H 9300 4350 60  0001 C CNN
+F 4 "C141311" H 9300 4250 50  0001 C CNN "LCSC Part"
 	1    9300 4250
 	-1   0    0    -1
