File: Clk.sch (KiCad schematic (older format))
At the start: 6 parts, among them U4 20M, U5 25M

Commit message: Moving toward new update system
Parts:
- C5, C6: LCSC Part (none) -> C23630
- R1, R2: value 22 -> 47; LCSC Part (none) -> C23182
- U4: LCSC Part (none) -> C32529
- U5: LCSC Part (none) -> C32526
Changed lines of the file:
@@
 AR Path="/61A87B62/6141AC14" Ref="R?"  Part="1"
 F 0 "R2" V 3600 2650 50  0000 C CNN
-F 1 "22" V 3700 2650 50  0000 C BNN
+F 1 "47" V 3700 2650 50  0000 C BNN
 F 2 "stdpads:R_0603" H 3750 2650 50  0001 C CNN
 F 3 "~" H 3750 2650 50  0001 C CNN
+F 4 "C23182" H 3750 2650 50  0001 C CNN "LCSC Part"
 	1    3750 2650
 	0    1    1    0
@@
 AR Path="/61A87B62/6141A918" Ref="R?"  Part="1"
 F 0 "R1" V 3600 2350 50  0000 C CNN
-F 1 "22" V 3700 2350 50  0000 C BNN
+F 1 "47" V 3700 2350 50  0000 C BNN
 F 2 "stdpads:R_0603" H 3750 2350 50  0001 C CNN
 F 3 "~" H 3750 2350 50  0001 C CNN
+F 4 "C23182" H 3750 2350 50  0001 C CNN "LCSC Part"
 	1    3750 2350
 	0    1    1    0
@@
 F 2 "stdpads:C_0603" H 3500 4250 50  0001 C CNN
 F 3 "~" H 3500 4250 50  0001 C CNN
+F 4 "C23630" H 3500 4250 50  0001 C CNN "LCSC Part"
 	1    3500 4250
 	1    0    0    -1
@@
 F 2 "stdpads:C_0603" H 3100 4250 50  0001 C CNN
 F 3 "~" H 3100 4250 50  0001 C CNN
+F 4 "C23630" H 3100 4250 50  0001 C CNN "LCSC Part"
 	1    3100 4250
 	1    0    0    -1
@@
 F 2 "stdpads:Crystal_SMD_3225-4Pin_3.2x2.5mm" H 4400 2250 50  0001 C CNN
 F 3 "" H 4400 2250 50  0001 C CNN
+F 4 "C32529" H 4400 2250 50  0001 C CNN "LCSC Part"
 	1    4400 2250
 	-1   0    0    -1
@@
 F 2 "stdpads:Crystal_SMD_3225-4Pin_3.2x2.5mm" H 4400 2750 50  0001 C CNN
 F 3 "" H 4400 2750 50  0001 C CNN
+F 4 "C32526" H 4400 2750 50  0001 C CNN "LCSC Part"
 	1    4400 2750
 	-1   0    0    -1
