File: Control.sch (KiCad schematic (older format))
At the start: 8 parts, among them U1 XC95144XL-TQ100

Commit message: Before I remove ESP32
Connections:
- net ~RESET~r: no longer names the net of U1.1 (I/O/GTS3)
- net ~RESET~r: no longer U1.99 (I/O/GSR)
- no-connect marks 0 -> 2
Changed lines of the file:
@@
 $Descr A4 11693 8268
 encoding utf-8
-Sheet 7 10
+Sheet 6 10
 Title ""
 Date ""
@@
 Text HLabel 8400 3700 0    50   Input ~ 0
 FCLK
-Text HLabel 8400 2400 0    50   Output ~ 0
-~RESET~r
 Text HLabel 10400 3100 2    50   Output ~ 0
 ADoutLE0
 Text HLabel 10400 3000 2    50   Output ~ 0
 ADoutLE1
-Text HLabel 8400 2300 0    50   Output ~ 0
-~RESET~r
 Text HLabel 8400 4800 0    50   Input ~ 0
 ~RESET~
@@
 Text HLabel 10400 5900 2    50   Output ~ 0
 TDO
+NoConn ~ 8400 2300
+NoConn ~ 8400 2400
 Wire Bus Line
 	10700 1400 10700 1800

Commit message: Moving toward new update system
Parts:
- C26, C27, C28, C29, C30, C31, C32: LCSC Part (none) -> C23630
- U1: LCSC Part (none) -> C45126
Connections:
- net SW2: now reaches U1.61 (P61)
Changed lines of the file:
@@
 F 2 "stdpads:C_0603" H 4700 7450 50  0001 C CNN
 F 3 "~" H 4700 7450 50  0001 C CNN
+F 4 "C23630" H 4700 7450 50  0001 C CNN "LCSC Part"
 	1    4700 7450
 	1    0    0    -1
@@
 F 2 "stdpads:C_0603" H 5100 7450 50  0001 C CNN
 F 3 "~" H 5100 7450 50  0001 C CNN
+F 4 "C23630" H 5100 7450 50  0001 C CNN "LCSC Part"
 	1    5100 7450
 	1    0    0    -1
@@
 F 2 "stdpads:C_0603" H 5500 7450 50  0001 C CNN
 F 3 "~" H 5500 7450 50  0001 C CNN
+F 4 "C23630" H 5500 7450 50  0001 C CNN "LCSC Part"
 	1    5500 7450
 	1    0    0    -1
@@
 F 2 "stdpads:C_0603" H 4300 7450 50  0001 C CNN
 F 3 "~" H 4300 7450 50  0001 C CNN
+F 4 "C23630" H 4300 7450 50  0001 C CNN "LCSC Part"
 	1    4300 7450
 	1    0    0    -1
@@
 F 2 "stdpads:C_0603" H 6300 7450 50  0001 C CNN
 F 3 "~" H 6300 7450 50  0001 C CNN
+F 4 "C23630" H 6300 7450 50  0001 C CNN "LCSC Part"
 	1    6300 7450
 	1    0    0    -1
@@
 F 2 "stdpads:C_0603" H 5900 7450 50  0001 C CNN
 F 3 "~" H 5900 7450 50  0001 C CNN
+F 4 "C23630" H 5900 7450 50  0001 C CNN "LCSC Part"
 	1    5900 7450
 	1    0    0    -1
@@
 F 2 "stdpads:C_0603" H 6700 7450 50  0001 C CNN
 F 3 "~" H 6700 7450 50  0001 C CNN
+F 4 "C23630" H 6700 7450 50  0001 C CNN "LCSC Part"
 	1    6700 7450
 	1    0    0    -1
@@
 F 2 "stdpads:TQFP-100_14x14mm_P0.5mm" H 9400 3500 50  0001 C CNN
 F 3 "https://www.xilinx.com/support/documentation/data_sheets/ds056.pdf" H 9400 3500 50  0001 C CNN
+F 4 "C45126" H 9400 3500 50  0001 C CNN "LCSC Part"
 	1    9400 3500
 	1    0    0    -1
@@
 NoConn ~ 8400 2300
 NoConn ~ 8400 2400
+Text HLabel 10400 4300 2    50   Input ~ 0
+SW2
 Wire Bus Line
 	10700 1400 10700 1800
