File: MC68k.sch (KiCad schematic (older format))
At the start: 3 parts, among them U14 MC68HC000FN20

Commit message: Moving toward new update system
Parts:
- C1, C2: LCSC Part (none) -> C15850
Changed lines of the file:
@@
 F 2 "stdpads:C_0805" H 1700 7300 50  0001 C CNN
 F 3 "~" H 1700 7300 50  0001 C CNN
+F 4 "C15850" H 1700 7300 50  0001 C CNN "LCSC Part"
 	1    1700 7300
 	1    0    0    -1
@@
 F 2 "stdpads:C_0805" H 1300 7300 50  0001 C CNN
 F 3 "~" H 1300 7300 50  0001 C CNN
+F 4 "C15850" H 1300 7300 50  0001 C CNN "LCSC Part"
 	1    1300 7300
 	1    0    0    -1
