File: PDS.sch (KiCad schematic (older format))
At the start: 6 parts, among them J1 MacSEPDS

Commit message: Moving toward new update system
Parts:
- C18, C19, C20, C22, C24: LCSC Part (none) -> C15850
Changed lines of the file:
@@
 F 2 "stdpads:C_0805" H 2100 6300 50  0001 C CNN
 F 3 "~" H 2100 6300 50  0001 C CNN
+F 4 "C15850" H 2100 6300 50  0001 C CNN "LCSC Part"
 	1    2100 6300
 	1    0    0    -1
@@
 F 2 "stdpads:C_0805" H 1700 6300 50  0001 C CNN
 F 3 "~" H 1700 6300 50  0001 C CNN
+F 4 "C15850" H 1700 6300 50  0001 C CNN "LCSC Part"
 	1    1700 6300
 	1    0    0    -1
@@
 F 2 "stdpads:C_0805" H 2900 6300 50  0001 C CNN
 F 3 "~" H 2900 6300 50  0001 C CNN
+F 4 "C15850" H 2900 6300 50  0001 C CNN "LCSC Part"
 	1    2900 6300
 	1    0    0    -1
@@
 F 2 "stdpads:C_0805" H 1300 6300 50  0001 C CNN
 F 3 "~" H 1300 6300 50  0001 C CNN
+F 4 "C15850" H 1300 6300 50  0001 C CNN "LCSC Part"
 	1    1300 6300
 	1    0    0    -1
@@
 F 2 "stdpads:C_0805" H 3700 6300 50  0001 C CNN
 F 3 "~" H 3700 6300 50  0001 C CNN
+F 4 "C15850" H 3700 6300 50  0001 C CNN "LCSC Part"
 	1    3700 6300
 	1    0    0    -1
