File: Power.sch (KiCad schematic (older format))
At the start: 8 parts, among them U3 AZ1117CH-3.3, U6 AZ1117CH2-3.3

Commit message: Moving toward new update system
Parts:
- C10, C3, C4, C7, C8, C9: LCSC Part (none) -> C15850
- U3: value AZ1117CH-3.3 -> AZ1117EH-3.3; LCSC Part (none) -> C108494
- U6: value AZ1117CH2-3.3 -> DNP-AZ1117CH2-3.3
Changed lines of the file:
@@
 P 5250 2100
 F 0 "U3" H 5250 2300 50  0000 C CNN
-F 1 "AZ1117CH-3.3" H 5250 2200 50  0000 C BNN
+F 1 "AZ1117EH-3.3" H 5250 2200 50  0000 C BNN
 F 2 "stdpads:SOT-223" H 5250 2300 50  0001 C CNN
 F 3 "http://www.diodes.com/datasheets/AP1117.pdf" H 5350 1850 50  0001 C CNN
+F 4 "C108494" H 5250 2100 50  0001 C CNN "LCSC Part"
 	1    5250 2100
 	1    0    0    -1
@@
 F 2 "stdpads:C_0805" H 4850 2250 50  0001 C CNN
 F 3 "~" H 4850 2250 50  0001 C CNN
+F 4 "C15850" H 4850 2250 50  0001 C CNN "LCSC Part"
 	1    4850 2250
 	1    0    0    -1
@@
 F 2 "stdpads:C_0805" H 5650 2250 50  0001 C CNN
 F 3 "~" H 5650 2250 50  0001 C CNN
+F 4 "C15850" H 5650 2250 50  0001 C CNN "LCSC Part"
 	1    5650 2250
 	-1   0    0    -1
@@
 F 2 "stdpads:C_0805" H 5650 3050 50  0001 C CNN
 F 3 "~" H 5650 3050 50  0001 C CNN
+F 4 "C15850" H 5650 3050 50  0001 C CNN "LCSC Part"
 	1    5650 3050
 	-1   0    0    -1
@@
 P 5250 2900
 F 0 "U6" H 5250 3100 50  0000 C CNN
-F 1 "AZ1117CH2-3.3" H 5250 3000 50  0000 C BNN
+F 1 "DNP-AZ1117CH2-3.3" H 5250 3000 50  0000 C BNN
 F 2 "stdpads:SOT-223" H 5250 3100 50  0001 C CNN
 F 3 "http://www.diodes.com/datasheets/AP1117.pdf" H 5350 2650 50  0001 C CNN
@@
 F 2 "stdpads:C_0805" H 4850 3050 50  0001 C CNN
 F 3 "~" H 4850 3050 50  0001 C CNN
+F 4 "C15850" H 4850 3050 50  0001 C CNN "LCSC Part"
 	1    4850 3050
 	1    0    0    -1
@@
 F 2 "stdpads:C_0805" H 6050 2250 50  0001 C CNN
 F 3 "~" H 6050 2250 50  0001 C CNN
+F 4 "C15850" H 6050 2250 50  0001 C CNN "LCSC Part"
 	1    6050 2250
 	-1   0    0    -1
@@
 F 2 "stdpads:C_0805" H 6050 3050 50  0001 C CNN
 F 3 "~" H 6050 3050 50  0001 C CNN
+F 4 "C15850" H 6050 3050 50  0001 C CNN "LCSC Part"
 	1    6050 3050
 	-1   0    0    -1
