File: Prog.sch (KiCad schematic (older format))
At the start: 35 parts, among them J2 JTAG, J3 USB_B_Micro, Q1 MMBT3904, Q2 MMBT3904, Q3 MMBT3904, Q4 MMBT3904, Q5 MMBT3904, U12 CH340G, U7 ESP32-PICO-D4, Y1 12M

Commit message: Moving toward new update system
Parts:
- removed C45: 10u, stdpads:C_0805, symbol Device:C_Small
- removed C50, C52, C53: 2u2, stdpads:C_0603, symbol Device:C_Small
- removed C51: 100n, stdpads:C_0603, symbol Device:C_Small
- removed Q3, Q4, Q5: MMBT3904, stdpads:SOT-23, symbol Transistor_BJT:MMBT3904
- removed R12: 22, stdpads:R_0603, symbol Device:R_Small
- removed R13, R14: 1k, stdpads:R_0603, symbol Device:R_Small
- removed R6, R7: 10k, stdpads:R_0603, symbol Device:R_Small
- removed U7: ESP32-PICO-D4, Package_DFN_QFN:QFN-48-1EP_7x7mm_P0.5mm_EP5.3x5.3mm_ThermalVias, symbol RF_Module:ESP32-PICO-D4
- added U7: 74AHCT573PW, stdpads:TSSOP-20_4.4x6.5mm_P0.65mm, symbol GW_Logic:74573
- C48: value 10u -> 22p; footprint stdpads:C_0805 -> stdpads:C_0603; LCSC Part (none) -> C1653
- J3: value USB_B_Micro -> microUSB; LCSC Part (none) -> C404969
- Q1, Q2: LCSC Part C20526 -> (none)
- R10: LCSC Part C25804 -> C21190
- R11, R8: value 10k -> 1k; LCSC Part C25804 -> C21190
- R5, R9: LCSC Part (none) -> C21190
- U12: LCSC Part (none) -> C14267
- Y1: footprint stdpads:Crystal_SMD_3225-4Pin_3.2x2.5mm -> stdpads:Crystal_HC49-SMD; symbol Device:Crystal_GND24_Small -> Device:Crystal_Small; LCSC Part C9002 -> C111117
Connections:
- net VDDSD is gone; now on net USB5V: C25.1
- net +3V3: now also R9.1; no longer C48.1, C49.1, R8.1
- net +5V: now also C49.1, R8.1, U7.11 (~LE~), U7.20 (Vcc); no longer R11.1
- net GND: now also U7.10 (GND), U7.2 (D0), U7.4 (D2), U7.6 (D4), U7.8 (D6), U7.9 (D7); no longer Y1.2, Y1.4
- net TCK: now also U7.14 (Q5)
- net TDI: now also U7.18 (Q1)
- net TDO: now also U12.9 (~CTS)
- net TMS: now also U7.16 (Q3)
- net USB5V: now also R11.2; no longer R9.1
- net ~RESET~: now also Q2.3 (C)
- net at C47.1, U12.7 (XI): now also Y1.2; no longer Y1.3
- net UTCK: now reaches U12.2 (TXD)
- net UTCK: now also U7.7 (D5)
- net at U12.3 (RXD): now also R9.2
- net at Q1.1 (B), R10.1: now also C48.1, Q2.1 (B), R11.1; no longer R9.2
- net DTR renamed UTDI
- net UTDI: now also U7.3 (D1)
- net EN renamed JTAG~OE~
- net JTAG~OE~: now also Q1.3 (C), U7.1 (~OE~); no longer Q2.3 (C)
- net RTS renamed UTMS
- net UTMS: now also U7.5 (D3)
- no-connect marks 4 -> 12
Other:
- note removed: "ESP32 serial download mode thingy"
- moved on the sheet: C11, C21, C23, C25, J2, R15, R16, R5, U12
