File: RAMROM.sch (KiCad schematic (older format))
At the start: 10 parts, among them U10 39SF040, U11 39SF040, U8 KM48C2100, U9 KM48C2100

Commit message: Moving toward new update system
Parts:
- C12, C13, C14, C15, C16, C17: value 2u2 -> 10u; LCSC Part (none) -> C15850
- U10, U11: LCSC Part (none) -> C72257
Changed lines of the file:
@@
 AR Path="/5F723900/61609D38" Ref="C13"  Part="1"
 F 0 "C13" H 5000 4700 50  0000 L CNN
-F 1 "2u2" H 5000 4600 50  0000 L CNN
+F 1 "10u" H 5000 4600 50  0000 L CNN
 F 2 "stdpads:C_0805" H 4950 4650 50  0001 C CNN
 F 3 "~" H 4950 4650 50  0001 C CNN
+F 4 "C15850" H 4950 4650 50  0001 C CNN "LCSC Part"
 	1    4950 4650
 	1    0    0    -1
@@
 AR Path="/5F723900/61609D3F" Ref="C12"  Part="1"
 F 0 "C12" H 4600 4700 50  0000 L CNN
-F 1 "2u2" H 4600 4600 50  0000 L CNN
+F 1 "10u" H 4600 4600 50  0000 L CNN
 F 2 "stdpads:C_0805" H 4550 4650 50  0001 C CNN
 F 3 "~" H 4550 4650 50  0001 C CNN
+F 4 "C15850" H 4550 4650 50  0001 C CNN "LCSC Part"
 	1    4550 4650
 	1    0    0    -1
@@
 AR Path="/5F723900/6160B1A0" Ref="C14"  Part="1"
 F 0 "C14" H 5400 4700 50  0000 L CNN
-F 1 "2u2" H 5400 4600 50  0000 L CNN
+F 1 "10u" H 5400 4600 50  0000 L CNN
 F 2 "stdpads:C_0805" H 5350 4650 50  0001 C CNN
 F 3 "~" H 5350 4650 50  0001 C CNN
+F 4 "C15850" H 5350 4650 50  0001 C CNN "LCSC Part"
 	1    5350 4650
 	1    0    0    -1
@@
 AR Path="/5F723900/6160C7C7" Ref="C15"  Part="1"
 F 0 "C15" H 5800 4700 50  0000 L CNN
-F 1 "2u2" H 5800 4600 50  0000 L CNN
+F 1 "10u" H 5800 4600 50  0000 L CNN
 F 2 "stdpads:C_0805" H 5750 4650 50  0001 C CNN
 F 3 "~" H 5750 4650 50  0001 C CNN
+F 4 "C15850" H 5750 4650 50  0001 C CNN "LCSC Part"
 	1    5750 4650
 	1    0    0    -1
@@
 F 2 "stdpads:PLCC-32" H 8700 1250 50  0001 C CNN
 F 3 "http://ww1.microchip.com/downloads/en/DeviceDoc/20005022C.pdf" H 8700 2300 50  0001 C CNN
+F 4 "C72257" H 8700 2300 50  0001 C CNN "LCSC Part"
 	1    8700 2300
 	1    0    0    -1
@@
 F 2 "stdpads:PLCC-32" H 8700 3450 50  0001 C CNN
 F 3 "http://ww1.microchip.com/downloads/en/DeviceDoc/20005022C.pdf" H 8700 4500 50  0001 C CNN
+F 4 "C72257" H 8700 4500 50  0001 C CNN "LCSC Part"
 	1    8700 4500
 	1    0    0    -1
@@
 AR Path="/5F723900/618714E1" Ref="C17"  Part="1"
 F 0 "C17" H 10500 4350 50  0000 L CNN
-F 1 "2u2" H 10500 4250 50  0000 L CNN
+F 1 "10u" H 10500 4250 50  0000 L CNN
 F 2 "stdpads:C_0805" H 10450 4300 50  0001 C CNN
 F 3 "~" H 10450 4300 50  0001 C CNN
+F 4 "C15850" H 10450 4300 50  0001 C CNN "LCSC Part"
 	1    10450 4300
 	1    0    0    -1
@@
 AR Path="/5F723900/618714E8" Ref="C16"  Part="1"
 F 0 "C16" H 10100 4350 50  0000 L CNN
-F 1 "2u2" H 10100 4250 50  0000 L CNN
+F 1 "10u" H 10100 4250 50  0000 L CNN
 F 2 "stdpads:C_0805" H 10050 4300 50  0001 C CNN
 F 3 "~" H 10050 4300 50  0001 C CNN
+F 4 "C15850" H 10050 4300 50  0001 C CNN "LCSC Part"
 	1    10050 4300
 	1    0    0    -1
 $EndComp
 $Comp
-L power:GND #PWR0150
+L power:GND #PWR0200
 U 1 1 618714EE
 P 10450 4400
-AR Path="/5F723900/618714EE" Ref="#PWR0150"  Part="1"
+AR Path="/5F723900/618714EE" Ref="#PWR0200"  Part="1"
 AR Path="/60D70CB4/618714EE" Ref="#PWR?"  Part="1"
-F 0 "#PWR0150" H 10450 4150 50  0001 C CNN
+F 0 "#PWR0200" H 10450 4150 50  0001 C CNN
 F 1 "GND" H 10450 4250 50  0000 C CNN
 F 2 "" H 10450 4400 50  0001 C CNN
