File: Warp-SE.kicad_pcb (KiCad board)
At the start: 4 copper layers, 109.1 x 102.1 mm, 112 parts, among them J1 MacSEPDS, J2 JTAG, J3 USB_B_Micro, Q1 MMBT3904, Q2 MMBT3904, Q3 MMBT3904, Q4 MMBT3904, Q5 MMBT3904, SW1 OSCSEL, U1 XC95144XL-TQ100, U10 39SF040, U11 39SF040, U12 CH340G, U13 74AHCT573, U14 MC68HC000FN20, U15 74AHCT573, U16 74AHCT573, U17 74AHCT573, U18 74AHCT573, U19 74AHCT573, U2 74AHCT573, U20 74AHCT573, U21 74AHCT573, U22 74AHCT573, U23 74AHCT573, U24 74AHCT573, U3 AZ1117CH-3.3, U4 20M, U5 25M, U6 AZ1117CH2-3.3, U7 ESP32-PICO-D4, U8 KM48C2100, U9 KM48C2100, Y1 12M

Commit message: Moving toward new update system
Parts:
- removed C45: 10u, stdpads:C_0805
- removed C50, C52, C53: 2u2, stdpads:C_0603
- removed C51: 100n, stdpads:C_0603
- removed the Q2 at (194.7, 65.5)
- removed Q3, Q4: MMBT3904, stdpads:SOT-23
- removed R12: 22, stdpads:R_0603
- removed R13, R14: 1k, stdpads:R_0603
- removed R7: 10k, stdpads:R_0603
- C12, C13, C14, C15, C16, C17: value 2u2 -> 10u
- C48: value 10u -> 22p; footprint stdpads:C_0805 -> stdpads:C_0603
- J3: value USB_B_Micro -> microUSB
- R1, R2: value 22 -> 47
- R11, R8: value 10k -> 1k
- SW1: footprint stdpads:SW_DIP_SPSTx02_Slide_DSHP02TS_P1.27mm -> stdpads:SW_DIP_SPSTx03_Slide_DSHP03TS_P1.27mm
- U13, U15, U16, U17, U18, U19, U2, U20, U21, U22, U23, U24: value 74AHCT573 -> 74AHCT573PW
- U3: value AZ1117CH-3.3 -> AZ1117EH-3.3
- U6: value AZ1117CH2-3.3 -> DNP-AZ1117CH2-3.3
- U7: value ESP32-PICO-D4 -> 74AHCT573PW; footprint Package_DFN_QFN:QFN-48-1EP_7x7mm_P0.5mm_EP5.3x5.3mm_ThermalVias -> stdpads:TSSOP-20_4.4x6.5mm_P0.65mm
- Y1: footprint stdpads:Crystal_SMD_3225-4Pin_3.2x2.5mm -> stdpads:Crystal_HC49-SMD
- moved R6 80.2 mm to (105.0, 113.8), turned to 270 degrees
- moved C11 67.6 mm to (121.8, 58.5), turned to 270 degrees
- moved C48 64.8 mm to (195.4, 109.0), turned to 180 degrees
- moved Q1 31.6 mm to (168.2, 42.1), turned to 270 degrees
- moved C47 29.7 mm to (191.1, 53.9)
- moved Y1 28.2 mm to (191.8, 46.3), turned to 270 degrees
- moved C46 25.6 mm to (188.4, 41.9), turned to 90 degrees
- moved R8 21.7 mm to (171.9, 41.0), turned to 180 degrees
- moved C25 20.0 mm to (196.2, 40.4)
- moved C49 16.6 mm to (176.3, 41.0)
- moved C21 16.4 mm to (181.0, 55.0)
- moved U7 11.9 mm to (174.1, 45.5), turned to 270 degrees
- moved U12 11.9 mm to (182.8, 48.9), turned to 90 degrees
- moved R5 9.23 mm to (184.0, 55.0)
- moved R9 7.95 mm to (186.9, 55.0)
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- renumbered Q5 to Q2
Connections:
- net /Prog/ETMS renamed Net-(U7-Pad15)
- C25 pad 1: /Prog/VDDSD -> /Prog/USB5V
- C48 pad 1: +3V3 -> Net-(C48-Pad1)
- C49 pad 1: +3V3 -> +5V
- Q1 pad 1: Net-(Q1-Pad1) -> Net-(C48-Pad1)
- Q1 pad 3: Net-(Q1-Pad3) -> /Prog/JTAG~OE~
- Q2 pad 1: Net-(Q5-Pad1) -> Net-(C48-Pad1)
- Q2 pad 3: Net-(Q5-Pad3) -> /Control/~RESET~
- R10 pad 1: Net-(Q1-Pad1) -> Net-(C48-Pad1)
- R11 pad 1: +5V -> Net-(C48-Pad1)
- R11 pad 2: Net-(Q1-Pad3) -> /Prog/USB5V
- R3 pad 1: +3V3 -> +5V
- R4 pad 1: +3V3 -> +5V
- R6 pad 1: /Prog/DTR -> +5V
- R6 pad 2: Net-(Q3-Pad1) -> /Control/SW2
- R8 pad 1: +3V3 -> +5V
- R8 pad 2: /Prog/EN -> /Prog/JTAG~OE~
- R9 pad 1: /Prog/USB5V -> +3V3
- R9 pad 2: Net-(Q1-Pad1) -> Net-(R9-Pad2)
- SW1 pad 3: GND -> /Control/SW2
- U1 pad 61: Net-(U1-Pad61) -> /Control/SW2
- U12 pad 13: /Prog/DTR -> /Prog/UTDI
- U12 pad 14: /Prog/RTS -> /Prog/UTMS
- U12 pad 2: Net-(U12-Pad2) -> /Prog/UTCK
- U12 pad 3: Net-(U12-Pad3) -> Net-(R9-Pad2)
- U12 pad 9: Net-(U12-Pad9) -> /Control/TDO
- U7 pad 1: +3V3 -> /Prog/JTAG~OE~
- U7 pad 10: Net-(U7-Pad10) -> GND
- U7 pad 11: /Control/TDO -> +5V
- U7 pad 12: /Control/TCK -> Net-(U7-Pad12)
- U7 pad 13: /Control/TDI -> Net-(U7-Pad13)
- U7 pad 14: /Control/TMS -> /Control/TCK
- U7 pad 16: /Prog/ETDI -> /Control/TMS
- U7 pad 18: Net-(U7-Pad18) -> /Control/TDI
- U7 pad 19: +3V3 -> Net-(U7-Pad19)
- U7 pad 2: Net-(U7-Pad2) -> GND
- U7 pad 20: /Prog/ETCK -> +5V
- U7 pad 3: +3V3 -> /Prog/UTDI
- U7 pad 4: +3V3 -> GND
- U7 pad 5: Net-(U7-Pad5) -> /Prog/UTMS
- U7 pad 6: Net-(U7-Pad6) -> GND
- U7 pad 7: Net-(U7-Pad7) -> /Prog/UTCK
- U7 pad 8: Net-(U7-Pad8) -> GND
- U7 pad 9: /Prog/EN -> GND
- Y1 pad 2: GND -> Net-(C47-Pad1)
Routing:
- net Net-(C48-Pad1): track 0.00 -> 99.3 mm, vias 0 -> 4
- net +3V3: track 495.2 -> 404.4 mm, vias 36 -> 23
- net Net-(Q5-Pad1): track 74.3 -> 0.00 mm, vias 5 -> 0
- net /Prog/EN: track 71.8 -> 0.00 mm, vias 3 -> 0
- net /Prog/RESET: track 42.8 -> 0.00 mm, vias 2 -> 0
- net /Control/~RESET~r: track 38.2 -> 0.00 mm, vias 1 -> 0
- net /Prog/IO0: track 36.5 -> 0.00 mm, vias 2 -> 0
- net Net-(U12-Pad3): track 29.1 -> 0.00 mm, vias 2 -> 0
- net /Prog/DTR: track 27.2 -> 0.00 mm, vias 2 -> 0
- net Net-(U12-Pad2): track 26.6 -> 0.00 mm, vias 2 -> 0
- net /Control/TCK: track 150.6 -> 127.3 mm
- net /Prog/RTS: track 22.6 -> 0.00 mm, vias 2 -> 0
- net /Control/SW2: track 0.00 -> 21.6 mm, vias 0 -> 3
- net /Control/TDI: track 162.9 -> 141.9 mm
- net /Control/TMS: track 150.5 -> 132.1 mm
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Other:
- board text added: "Fast ROM"
- board text added: "Mac ROM"
- board text added: "WarpSE"
- board text removed: "Warp-SE"
