File: Warp-SE.kicad_sch (KiCad schematic)
At the start: 9 parts

Commit message: Migrate to KiCAD 6
Changed lines of the file:
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@@
   (junction (at 71.12 59.69) (diameter 0) (color 0 0 0 0)
   )
-  (junction (at 134.62 88.9) (diameter 0) (color 0 0 0 0)
-  )
   (junction (at 71.12 68.58) (diameter 0) (color 0 0 0 0)
   )
@@
   (junction (at 78.74 40.64) (diameter 0) (color 0 0 0 0)
   )
+  (junction (at 134.62 93.98) (diameter 0) (color 0 0 0 0)
+  )
   (bus (pts (xy 71.12 27.94) (xy 71.12 59.69))
     (stroke (width 0) (type default) (color 0 0 0 0))
@@
     (stroke (width 0) (type default) (color 0 0 0 0))
   )
-  (wire (pts (xy 134.62 67.31) (xy 134.62 88.9))
-    (stroke (width 0) (type default) (color 0 0 0 0))
-  )
   (bus (pts (xy 40.64 78.74) (xy 43.18 78.74))
     (stroke (width 0) (type default) (color 0 0 0 0))
@@
     (stroke (width 0) (type default) (color 0 0 0 0))
   )
-  (wire (pts (xy 119.38 73.66) (xy 106.68 73.66))
-    (stroke (width 0) (type default) (color 0 0 0 0))
-  )
   (wire (pts (xy 40.64 48.26) (xy 81.28 48.26))
     (stroke (width 0) (type default) (color 0 0 0 0))
@@
     (stroke (width 0) (type default) (color 0 0 0 0))
   )
-  (wire (pts (xy 134.62 88.9) (xy 106.68 88.9))
+  (wire (pts (xy 106.68 88.9) (xy 137.16 88.9))
     (stroke (width 0) (type default) (color 0 0 0 0))
   )
@@
     (stroke (width 0) (type default) (color 0 0 0 0))
   )
+  (wire (pts (xy 134.62 67.31) (xy 134.62 93.98))
+    (stroke (width 0) (type default) (color 0 0 0 0))
+  )
   (wire (pts (xy 33.02 176.53) (xy 25.4 176.53))
     (stroke (width 0) (type default) (color 0 0 0 0))
@@
     (stroke (width 0) (type default) (color 0 0 0 0))
   )
+  (wire (pts (xy 134.62 93.98) (xy 137.16 93.98))
+    (stroke (width 0) (type default) (color 0 0 0 0))
+  )
   (bus (pts (xy 71.12 68.58) (xy 68.58 68.58))
     (stroke (width 0) (type default) (color 0 0 0 0))
@@
     (stroke (width 0) (type default) (color 0 0 0 0))
   )
-  (wire (pts (xy 137.16 88.9) (xy 134.62 88.9))
-    (stroke (width 0) (type default) (color 0 0 0 0))
-  )
   (wire (pts (xy 114.3 59.69) (xy 137.16 59.69))
     (stroke (width 0) (type default) (color 0 0 0 0))
@@
     (stroke (width 0) (type default) (color 0 0 0 0))
   )
-  (wire (pts (xy 106.68 93.98) (xy 137.16 93.98))
+  (wire (pts (xy 106.68 93.98) (xy 134.62 93.98))
     (stroke (width 0) (type default) (color 0 0 0 0))
   )
@@
       (reference "R4") (unit 1) (value "10k") (footprint "stdpads:R_0603")
     )
-    (path "/00000000-0000-0000-0000-000061aa52c4/00000000-0000-0000-0000-000061afea26"
-      (reference "R5") (unit 1) (value "1k") (footprint "stdpads:R_0603")
+    (path "/00000000-0000-0000-0000-000061aa52c4/46a0a607-6113-4fdf-ba11-cbd5f8cadd3f"
+      (reference "R5") (unit 1) (value "10k") (footprint "stdpads:R_0603")
     )
     (path "/00000000-0000-0000-0000-000061a87b62/00000000-0000-0000-0000-000061e3af0c"
       (reference "R6") (unit 1) (value "10k") (footprint "stdpads:R_0603")
     )
-    (path "/00000000-0000-0000-0000-000061aa52c4/00000000-0000-0000-0000-000061f500b1"
-      (reference "R8") (unit 1) (value "1k") (footprint "stdpads:R_0603")
-    )
-    (path "/00000000-0000-0000-0000-000061aa52c4/00000000-0000-0000-0000-0000621fd768"
-      (reference "R9") (unit 1) (value "1k") (footprint "stdpads:R_0603")
-    )
-    (path "/00000000-0000-0000-0000-000061aa52c4/00000000-0000-0000-0000-000061f022fd"
-      (reference "R10") (unit 1) (value "1k") (footprint "stdpads:R_0603")
+    (path "/00000000-0000-0000-0000-000061aa52c4/5e6c5236-5da5-4208-91c5-fc14b0b86117"
+      (reference "R8") (unit 1) (value "10k") (footprint "stdpads:R_0603")
+    )
+    (path "/00000000-0000-0000-0000-000061aa52c4/9d1ef6fd-6f67-4e97-87be-f7bbf4ac7873"
+      (reference "R9") (unit 1) (value "10k") (footprint "stdpads:R_0603")
+    )
+    (path "/00000000-0000-0000-0000-000061aa52c4/43161de2-4bad-47e3-b719-fe3b7aecf870"
+      (reference "R10") (unit 1) (value "10k") (footprint "stdpads:R_0603")
     )
     (path "/00000000-0000-0000-0000-000061aa52c4/00000000-0000-0000-0000-000061f02307"
-      (reference "R11") (unit 1) (value "1k") (footprint "stdpads:R_0603")
+      (reference "R11") (unit 1) (value "10k") (footprint "stdpads:R_0603")
     )
     (path "/00000000-0000-0000-0000-000061aa52c4/00000000-0000-0000-0000-000062762b96"
@@
       (reference "R16") (unit 1) (value "10k") (footprint "stdpads:R_0603")
     )
+    (path "/00000000-0000-0000-0000-000061aa52c4/2d3f37d7-6080-4b18-978b-5047c1658a26"
+      (reference "R?") (unit 1) (value "10k") (footprint "stdpads:R_0603")
+    )
     (path "/00000000-0000-0000-0000-000061a87b62/00000000-0000-0000-0000-000061a8bbd9"
