File: CPUBuf.kicad_sch (KiCad schematic)
At the start: 6 parts

Commit message: Switch to '030
Parts:
- removed U? (x4): 74LVC245APW, symbol GW_Logic:74245
- removed U?: 74245, symbol GW_Logic:74245
- added U? (x8): 74LVC245APW, symbol GW_Logic:74245
- U?: value 74245 -> 74LVC245APW
Connections:
- net MD31: now reaches U?.2 (A0)
- net MD30: now reaches U?.3 (A1)
- net MD29: now reaches U?.4 (A2)
- net MD28: now reaches U?.5 (A3)
- net MD27: now reaches U?.6 (A4)
- net MD26: now reaches U?.7 (A5)
- net MD25: now reaches U?.8 (A6)
- net MD24: now reaches U?.9 (A7)
- new net CA0: U?.2 (A0)
- new net CA1: U?.3 (A1)
- new net CA10: U?.9 (A7)
- new net CA11: U?.8 (A6)
- new net CA12: U?.7 (A5)
- new net CA13: U?.6 (A4)
- new net CA14: U?.5 (A3)
- new net CA15: U?.4 (A2)
- new net CA16: U?.3 (A1)
- new net CA17: U?.2 (A0)
- new net CA18: U?.9 (A7)
- new net CA19: U?.8 (A6)
- new net CA2: U?.9 (A7)
- new net CA20: U?.7 (A5)
- new net CA21: U?.6 (A4)
- new net CA22: U?.5 (A3)
- new net CA23: U?.4 (A2)
- new net CA24: U?.9 (A7)
- new net CA3: U?.8 (A6)
- new net CA31: U?.8 (A6)
- new net CA4: U?.7 (A5)
- new net CA5: U?.6 (A4)
- new net CA6: U?.5 (A3)
- new net CA7: U?.4 (A2)
- new net CA8: U?.3 (A1)
- new net CA9: U?.2 (A0)
- new net CFC0: U?.8 (A6)
- new net CFC1: U?.7 (A5)
- new net CFC2: U?.6 (A4)
- new net CR~{W}: U?.3 (A1)
- new net CSIZ0: U?.5 (A3)
- new net CSIZ1: U?.4 (A2)
- new net C~{AS}: U?.2 (A0)
- new net C~{BG}: U?.6 (A4)
- new net C~{CBREQ}: U?.7 (A5)
- new net C~{CIOUT}: U?.9 (A7)
- new net FA0: U?.18 (B0)
- new net FA1: U?.17 (B1)
- new net FA10: U?.11 (B7)
- new net FA11: U?.12 (B6)
- new net FA12: U?.13 (B5)
- new net FA13: U?.14 (B4)
- new net FA14: U?.15 (B3)
- new net FA15: U?.16 (B2)
- new net FA16: U?.17 (B1)
- new net FA17: U?.18 (B0)
- new net FA18: U?.11 (B7)
- new net FA19: U?.12 (B6)
- new net FA2: U?.11 (B7)
- new net FA20: U?.13 (B5)
- new net FA21: U?.14 (B4)
- new net FA22: U?.15 (B3)
- new net FA23: U?.16 (B2)
- new net FA24: U?.11 (B7)
- new net FA3: U?.12 (B6)
- new net FA31: U?.12 (B6)
- new net FA4: U?.13 (B5)
- new net FA5: U?.14 (B4)
- new net FA6: U?.15 (B3)
- new net FA7: U?.16 (B2)
- new net FA8: U?.17 (B1)
- new net FA9: U?.18 (B0)
- new net FFC0: U?.12 (B6)
- new net FFC1: U?.13 (B5)
- new net FFC2: U?.14 (B4)
- new net FR~{W}: U?.17 (B1)
- new net FSIZ0: U?.15 (B3)
- new net FSIZ1: U?.16 (B2)
- new net F~{AS}: U?.18 (B0)
- new net F~{BG}: U?.14 (B4)
- new net F~{CBREQ}: U?.13 (B5)
- new net F~{CIOUT}: U?.11 (B7)
- new net MD0: U?.9 (A7)
- new net MD1: U?.8 (A6)
- new net MD10: U?.7 (A5)
- new net MD11: U?.6 (A4)
- new net MD12: U?.5 (A3)
- new net MD13: U?.4 (A2)
- new net MD14: U?.3 (A1)
- new net MD15: U?.2 (A0)
- new net MD16: U?.9 (A7)
- new net MD17: U?.8 (A6)
- new net MD18: U?.7 (A5)
- new net MD19: U?.6 (A4)
- new net MD2: U?.7 (A5)
- new net MD20: U?.5 (A3)
- new net MD21: U?.4 (A2)
- new net MD22: U?.3 (A1)
- new net MD23: U?.2 (A0)
- new net MD3: U?.6 (A4)
- new net MD4: U?.5 (A3)
- new net MD5: U?.4 (A2)
- new net MD6: U?.3 (A1)
- new net MD7: U?.2 (A0)
- new net MD8: U?.9 (A7)
- new net MD9: U?.8 (A6)
