File: WarpSE.kicad_pcb (KiCad board)
At the start: 4 copper layers, 109.1 x 102.1 mm, 42 parts, among them J1 MacSEPDS, J2 JTAG, J3 microUSB, Q1 MMBT3904, Q2 MMBT3904, U12 CH340G, U13 74AHCT573PW, U15 74AHCT573PW, U16 74AHCT573PW, U19 74AHCT573PW, U21 74AHCT573PW, U7 74AHCT573PW, Y1 12M

Commit message: more
Parts:
- removed J2: JTAG, Connector:Tag-Connect_TC2050-IDC-FP_2x05_P1.27mm_Vertical
- removed R15: 10k, stdpads:R_0603
- added C35: 2u2, stdpads:C_0603, F.Cu at (190.3, 57.9)
- added C44: 2u2, stdpads:C_0603, F.Cu at (190.3, 116.2)
- added C44: 2u2, stdpads:C_0603, F.Cu at (180.3, 116.2)
- added REF**: TSOP-II-54_22.2x10.16mm_P0.8mm, stdpads:TSOP-II-54_22.2x10.16mm_P0.8mm, F.Cu at (157.5, 101.5)
- added U13: 74AHCT573PW, stdpads:TSSOP-20_4.4x6.5mm_P0.65mm, F.Cu at (178.1, 120.5)
- added U13: 74AHCT573PW, stdpads:TSSOP-20_4.4x6.5mm_P0.65mm, F.Cu at (188.1, 120.5)
- added U21: 74AHCT573PW, stdpads:TSSOP-20_4.4x6.5mm_P0.65mm, F.Cu at (188.1, 62.3)
- moved FID1 29.2 mm to (134.5, 42.4)
- moved H1 29.2 mm to (134.5, 39.9)
- moved REF** 17.9 mm to (157.5, 76.5), turned to 180 degrees
- moved C42 9.10 mm to (190.3, 94.3)
- moved U15 9.10 mm to (188.1, 98.7)
- moved C40 9.10 mm to (190.3, 85.2)
- moved C44 9.10 mm to (190.3, 103.5)
- moved U13 9.10 mm to (188.1, 107.8)
- moved U16 9.10 mm to (188.1, 89.6)
- moved C48 6.85 mm to (195.4, 102.2)
- moved Q2 6.85 mm to (195.2, 105.0)
Routing:
- net /Prog/TDO: track 156.3 -> 19.0 mm, vias 3 -> 1
- net /Control/C16M: track 93.7 -> 0.00 mm
- net /Control/C8M: track 88.1 -> 0.00 mm
- net /Control/MacE: track 82.6 -> 0.00 mm
- net +3V3: track 170.0 -> 90.7 mm, vias 7 -> 6
- net /Control/TDI: track 85.9 -> 11.6 mm, vias 2 -> 1
- net /Control/Mac~{BERR}: track 77.8 -> 3.96 mm
- net /Control/TMS: track 81.9 -> 12.2 mm, vias 2 -> 1
- net /Control/TCK: track 78.1 -> 13.0 mm, vias 2 -> 1
- net Net-(C48-Pad1): track 56.0 -> 10.9 mm
- net /Control/U~{WE}: track 44.0 -> 0.00 mm
- net /Buf/MacA23: track 40.0 -> 12.7 mm
- net /Buf/MacA22: track 38.0 -> 12.8 mm
- net /Buf/MacA21: track 36.1 -> 12.8 mm
- net /Buf/MacA16: track 31.4 -> 9.34 mm
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Other:
- board size 109.1 x 102.1 mm -> 79.9 x 102.1 mm
- board text removed: "4410A"
- board text removed: "Accelerator for Mac SE"
- board text removed: "GW"
- board text removed: "Garrett’s Workshop"
- board text removed: "WarpSE"

Commit message: more
Parts:
- added G***: LOGO, LOGO, F.Cu at (146.6, 51.2)
- added G***: LOGO, LOGO, F.Cu at (146.6, 44.8)
Routing:
- net /Control/Mac~{BERR}: track 3.96 -> 59.9 mm, vias 0 -> 1
- net /Control/C16M: track 0.00 -> 14.8 mm
- net /Control/MacE: track 0.00 -> 13.8 mm
- net /Control/C8M: track 0.00 -> 13.6 mm
- net GND: vias 222 -> 221

Commit message: idk
Parts:
- removed C18, C20, C24: 10u, stdpads:C_0805
- removed C23, C25, C35 (x2), C37, C40, C42, C44 (x3), C49: 2u2, stdpads:C_0603
- removed C46, C47, C48: 22p, stdpads:C_0603
- removed the G*** at (146.6, 51.2)
- removed the G*** at (146.6, 44.8)
- removed Q1, Q2: MMBT3904, stdpads:SOT-23
- removed R10, R11, R7, R8, R9: 10k, stdpads:R_0603
- removed the REF** at (157.5, 76.5)
- removed U12: CH340G, stdpads:SOIC-16_3.9mm
- removed U13 (x3), U15, U16, U19, U21 (x2), U7: 74AHCT573PW, stdpads:TSSOP-20_4.4x6.5mm_P0.65mm
- removed Y1: 12M, stdpads:Crystal_HC49-SMD
- added G***: LOGO, LOGO, F.Cu at (162.2, 51.6)
- added G***: LOGO, LOGO, F.Cu at (162.2, 44.2)
- added REF**: SOT-353, stdpads:SOT-353, F.Cu at (193.1, 69.7)
- added REF**: R_0603, stdpads:R_0603, F.Cu at (177.4, 62.7)
- added REF**: TSSOP-20_4.4x6.5mm_P0.65mm, stdpads:TSSOP-20_4.4x6.5mm_P0.65mm, F.Cu at (190.7, 74.8)
- added REF**: R_0603, stdpads:R_0603, F.Cu at (177.3, 52.7)
- added REF**: SOT-353, stdpads:SOT-353, F.Cu at (193.1, 127.2)
- added REF**: TSSOP-20_4.4x6.5mm_P0.65mm, stdpads:TSSOP-20_4.4x6.5mm_P0.65mm, F.Cu at (190.7, 82.7)
- added REF**: TSSOP-20_4.4x6.5mm_P0.65mm, stdpads:TSSOP-20_4.4x6.5mm_P0.65mm, F.Cu at (190.7, 98.5)
- added REF**: TSSOP-20_4.4x6.5mm_P0.65mm, stdpads:TSSOP-20_4.4x6.5mm_P0.65mm, F.Cu at (190.7, 122.2)
- added REF**: R_0603, stdpads:R_0603, F.Cu at (185.8, 69.8)
- added REF**: C_0603, stdpads:C_0603, F.Cu at (194.9, 53.1)
- added REF**: TSSOP-20_4.4x6.5mm_P0.65mm, stdpads:TSSOP-20_4.4x6.5mm_P0.65mm, F.Cu at (190.7, 114.2)
- added REF**: Tag-Connect_TC2050-IDC-FP_2x05_P1.27mm_Vertical, stdpads:Tag-Connect_TC2050-IDC-FP_2x05_P1.27mm_Vertical, F.Cu at (161.5, 102.3)
- added REF**: Tag-Connect_TC2050-IDC-FP_2x05_P1.27mm_Vertical, stdpads:Tag-Connect_TC2050-IDC-FP_2x05_P1.27mm_Vertical, F.Cu at (161.2, 63.3)
- added REF**: TSSOP-20_4.4x6.5mm_P0.65mm, stdpads:TSSOP-20_4.4x6.5mm_P0.65mm, F.Cu at (190.7, 90.5)
- added REF**: SOIC-8_3.9mm, stdpads:SOIC-8_3.9mm, F.Cu at (177.5, 57.7)
- added REF**: R_0603, stdpads:R_0603, F.Cu at (173.0, 112.6)
- added REF**: C_0603, stdpads:C_0603, F.Cu at (194.9, 46.6)
- added REF**: R_0603, stdpads:R_0603, F.Cu at (152.5, 122.2)
- added REF**: SOIC-8_5.3mm, stdpads:SOIC-8_5.3mm, F.Cu at (169.4, 122.5)
- added REF**: TSSOP-20_4.4x6.5mm_P0.65mm, stdpads:TSSOP-20_4.4x6.5mm_P0.65mm, F.Cu at (190.7, 106.3)
- added REF**: SOT-353, stdpads:SOT-353, F.Cu at (188.3, 69.7)
- added REF**: SOIC-8_5.3mm, stdpads:SOIC-8_5.3mm, F.Cu at (158.5, 122.7)
- added REF**: C_0402, stdpads:C_0402, B.Cu at (187.7, 69.8)
- added REF**: C_0402, stdpads:C_0402, B.Cu at (178.7, 99.6)
- added REF**: C_0402, stdpads:C_0402, B.Cu at (176.4, 57.0)
- added REF**: C_0402, stdpads:C_0402, B.Cu at (172.6, 103.6)
- added REF**: C_0402, stdpads:C_0402, B.Cu at (191.9, 103.9)
- added REF**: C_0402, stdpads:C_0402, B.Cu at (177.6, 101.6)
- added REF**: C_0402, stdpads:C_0402, B.Cu at (188.3, 127.2)
- added REF**: C_0402, stdpads:C_0402, B.Cu at (191.9, 88.1)
- added REF**: C_0402, stdpads:C_0402, B.Cu at (178.7, 103.6)
- added REF**: C_0402, stdpads:C_0402, B.Cu at (191.9, 96.0)
- added REF**: R_0603, stdpads:R_0603, F.Cu at (175.3, 92.1)
- added REF**: C_0402, stdpads:C_0402, B.Cu at (176.8, 104.7)
- added REF**: C_0402, stdpads:C_0402, B.Cu at (159.8, 121.3)
- added REF**: C_0402, stdpads:C_0402, B.Cu at (174.4, 104.7)
- added REF**: C_0402, stdpads:C_0402, B.Cu at (175.6, 100.0)
- added REF**: C_0402, stdpads:C_0402, B.Cu at (186.5, 45.2)
- added REF**: C_0402, stdpads:C_0402, B.Cu at (191.9, 111.8)
- added REF**: C_0402, stdpads:C_0402, B.Cu at (174.4, 101.6)
- added REF**: C_0402, stdpads:C_0402, B.Cu at (191.9, 72.3)
- added REF**: C_0402, stdpads:C_0402, B.Cu at (192.2, 69.8)
- added REF**: C_0402, stdpads:C_0402, B.Cu at (170.9, 120.9)
- added REF**: SOIC-28_7.5mm, stdpads:SOIC-28_7.5mm, F.Cu at (186.5, 55.0)
- added REF**: C_0402, stdpads:C_0402, B.Cu at (174.4, 98.5)
- added REF**: C_0402, stdpads:C_0402, B.Cu at (191.9, 119.7)
- added REF**: C_0402, stdpads:C_0402, B.Cu at (172.3, 101.6)
- added REF**: C_0402, stdpads:C_0402, B.Cu at (172.6, 99.6)
- added REF**: C_0402, stdpads:C_0402, B.Cu at (193.1, 127.2)
- added REF**: C_0402, stdpads:C_0402, B.Cu at (176.8, 98.5)
- added REF**: C_0402, stdpads:C_0402, B.Cu at (175.6, 103.2)
- added REF**: C_0402, stdpads:C_0402, B.Cu at (191.9, 80.2)
- added REF**: R_0603, stdpads:R_0603, F.Cu at (175.9, 121.2)
- added REF**: Crystal_SMD_3225-4Pin_3.2x2.5mm, stdpads:Crystal_SMD_3225-4Pin_3.2x2.5mm, F.Cu at (195.0, 49.9)
- added REF**: SOT-353, stdpads:SOT-353, F.Cu at (188.3, 127.2)
- added REF**: R_0603, stdpads:R_0603, F.Cu at (192.8, 67.7)
- added U11: LFE5U-12F-BG256, stdpads:Lattice_CABGA-256_14x14mm, F.Cu at (175.6, 101.6)
- J3: footprint stdpads:USB_Micro-B_ShouHan_MicroXNJ -> stdpads:USB_Micro-B_Amphenol_10118192-0001
- moved REF** 25.2 mm to (173.4, 82.0), turned to 0 degrees
- moved H1 19.2 mm to (153.5, 42.0)
- moved FID1 16.5 mm to (151.0, 42.0)
- moved C22 15.1 mm to (209.6, 50.0)
- moved J3 3.62 mm to (186.5, 42.0), turned to 180 degrees
- moved FID2 2.16 mm to (207.8, 42.0)
- moved H2 2.16 mm to (210.3, 42.0)
Connections:
- net /Control/C16M renamed /PDS/C16M
- net /Control/C8M renamed /PDS/C8M
- net /Control/MacE renamed /PDS/E
- net /Control/Mac~{AS} renamed /PDS/~{AS}
- net /Control/Mac~{BERR} renamed /PDS/~{BERR}
- net /Control/Mac~{BR} renamed /PDS/~{BR}
- net /Control/Mac~{DTACK} renamed /PDS/~{DTACK}
- net /Control/Mac~{LDS} renamed /PDS/~{LDS}
- net /Control/Mac~{UDS} renamed /PDS/~{UDS}
- net /Control/Mac~{VMA} renamed /PDS/~{VMA}
- net /Control/Mac~{VPA} renamed /PDS/~{VPA}
- net /Control/~{IPL}2 renamed /Control/B~{IPL}2
- net /MC68k/~{IPL}0 renamed /Control/B~{IPL}0
- net /MC68k/~{IPL}1 renamed /Control/B~{IPL}1
- J1 pad A10: /Buf/MacA7 -> /PDS/A7
- J1 pad A11: /Buf/MacA8 -> /PDS/A8
- J1 pad A12: /Buf/MacA9 -> /PDS/A9
- J1 pad A13: /Buf/MacA10 -> /PDS/A10
- J1 pad A14: /Buf/MacA11 -> /PDS/A11
- J1 pad A15: /Buf/MacA12 -> /PDS/A12
- J1 pad A16: /Buf/MacA13 -> /PDS/A13
- J1 pad A17: /Buf/MacA14 -> /PDS/A14
- J1 pad A18: /Buf/MacA15 -> /PDS/A15
- J1 pad A19: /Buf/MacA16 -> /PDS/A16
- J1 pad A20: /Buf/MacA17 -> /PDS/A17
- J1 pad A21: /Buf/MacA18 -> /PDS/A18
- J1 pad A22: /Buf/MacA19 -> /PDS/A19
- J1 pad A23: /Buf/MacA20 -> /PDS/A20
- J1 pad A24: /Buf/MacA21 -> /PDS/A21
- J1 pad A25: /Buf/MacA22 -> /PDS/A22
- J1 pad A26: /Buf/MacA23 -> /PDS/A23
- J1 pad A4: /Buf/MacA1 -> /PDS/A1
- J1 pad A5: /Buf/MacA2 -> /PDS/A2
- J1 pad A6: /Buf/MacA3 -> /PDS/A3
- J1 pad A7: /Buf/MacA4 -> /PDS/A4
- J1 pad A8: /Buf/MacA5 -> /PDS/A5
- J1 pad A9: /Buf/MacA6 -> /PDS/A6
- J1 pad C12: /Control/~{RESET} -> /PDS/~{RESET}
- J1 pad C14: /Buf/MacD0 -> /PDS/D0
- J1 pad C15: /Buf/MacD1 -> /PDS/D1
- J1 pad C16: /Buf/MacD2 -> /PDS/D2
- J1 pad C17: /Buf/MacD3 -> /PDS/D3
- J1 pad C18: /Buf/MacD4 -> /PDS/D4
- J1 pad C19: /Buf/MacD5 -> /PDS/D5
- J1 pad C20: /Buf/MacD6 -> /PDS/D6
- J1 pad C21: /Buf/MacD7 -> /PDS/D7
- J1 pad C22: /Buf/MacD8 -> /PDS/D8
- J1 pad C23: /Buf/MacD9 -> /PDS/D9
- J1 pad C24: /Buf/MacD10 -> /PDS/D10
- J1 pad C25: /Buf/MacD11 -> /PDS/D11
- J1 pad C26: /Buf/MacD12 -> /PDS/D12
- J1 pad C27: /Buf/MacD13 -> /PDS/D13
- J1 pad C28: /Buf/MacD14 -> /PDS/D14
- J1 pad C29: /Buf/MacD15 -> /PDS/D15
- J1 pad C5: /Control/Mac~{BG} -> unconnected-(J1C-~{BG}-PadC5)
- J1 pad C7: /Buf/Mac~{R}W -> /PDS/R~{W}
Routing:
- net +3V3: track 90.7 -> 7.35 mm, vias 6 -> 13
- net /Control/B~{IPL}2: track 73.5 -> 0.00 mm
- net /Control/B~{IPL}1: track 69.4 -> 0.00 mm
- net /Control/B~{IPL}0: track 65.1 -> 0.00 mm
- net /PDS/~{BERR}: track 59.9 -> 0.00 mm, vias 1 -> 0
- net +5V: track 50.3 -> 0.00 mm, vias 42 -> 0
- net /Buf/ADoutLE0: track 47.1 -> 0.00 mm, vias 7 -> 0
- net GND: track 75.1 -> 28.4 mm, vias 221 -> 142
- net Net-(Q1-Pad1): track 42.2 -> 0.00 mm, vias 2 -> 0
- net /Prog/USB5V: track 37.7 -> 1.08 mm, vias 4 -> 1
- net /Control/~{RESET}: track 25.2 -> 0.00 mm, vias 1 -> 0
- net /Buf/MacA8: track 22.2 -> 0.00 mm
- net /Buf/Mac~{R}W: track 21.7 -> 0.00 mm, vias 1 -> 0
- net /Buf/Aout~{OE}: track 21.4 -> 0.00 mm, vias 3 -> 0
- net /Buf/MacA7: track 19.9 -> 0.00 mm
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Other:
- board size 79.9 x 102.1 mm -> 63.4 x 99.9 mm
- rule pad_to_mask_clearance: 0.05 -> 0.0762
- board text added: "ZK, GF"
