File: PDS.kicad_sch (KiCad schematic)
At the start: 6 parts, among them J1 MacSEPDS

Commit message: idk
Connections:
- net ~{BG}: no longer names the net of J1.C5 (~{BG})
- no-connect marks 16 -> 17
Changed lines of the file:
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@@
   (no_connect (at 102.87 66.04))
   (no_connect (at 72.39 81.28))
+  (no_connect (at 102.87 68.58))
   (no_connect (at 72.39 121.92))
   (no_connect (at 72.39 116.84))
@@
     (effects (font (size 1.27 1.27)) (justify left))
   )
-  (hierarchical_label "~{BG}" (shape output) (at 102.87 68.58 0) (fields_autoplaced)
-    (effects (font (size 1.27 1.27)) (justify left))
-  )
