File: PDS.kicad_sch (KiCad schematic)
At the start: 3 parts, among them J1 MacSEPDS

Commit message: Before switching to SiT2001 oscillator
Parts:
- removed R27: 680, stdpads:R_0805, symbol Device:R_Small
Changed lines of the file:
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@@
 	)
 	(junction
-		(at 43.18 162.56)
-		(diameter 0)
-		(color 0 0 0 0)
-	)
-	(junction
 		(at 72.39 93.98)
 		(diameter 0)
@@
 		)
 	)
-	(bus
+	(wire
 		(pts
-			(xy 45.72 109.22) (xy 45.72 111.76)
+			(xy 31.75 157.48) (xy 33.02 157.48)
 		)
 		(stroke
@@
 		)
 	)
-	(wire
+	(bus
 		(pts
-			(xy 33.02 157.48) (xy 43.18 157.48)
+			(xy 45.72 109.22) (xy 45.72 111.76)
 		)
 		(stroke
@@
 	(wire
 		(pts
-			(xy 33.02 162.56) (xy 43.18 162.56)
-		)
-		(stroke
-			(width 0)
-			(type default)
-		)
-	)
-	(wire
-		(pts
 			(xy 102.87 129.54) (xy 107.95 129.54)
 		)
@@
 	(global_label "+5Vin"
 		(shape input)
-		(at 33.02 157.48 180)
+		(at 31.75 157.48 180)
 		(fields_autoplaced yes)
 		(effects
@@
 		)
 		(property "Intersheetrefs" "${INTERSHEET_REFS}"
-			(at 25.0647 157.48 0)
+			(at 23.7947 157.48 0)
 			(effects
 				(font
@@
 	)
 	(symbol
-		(lib_id "power:GND")
-		(at 43.18 162.56 0)
-		(mirror y)
-		(unit 1)
-		(exclude_from_sim no)
-		(in_bom yes)
-		(on_board yes)
-		(dnp no)
-		(property "Reference" "#PWR0153"
-			(at 43.18 168.91 0)
-			(effects
-				(font
-					(size 1.27 1.27)
-				)
-				(hide yes)
-			)
-		)
-		(property "Value" "GND"
-			(at 43.18 166.37 0)
-			(effects
-				(font
-					(size 1.27 1.27)
-				)
-			)
-		)
-		(property "Footprint" ""
-			(at 43.18 162.56 0)
-			(effects
-				(font
-					(size 1.27 1.27)
-				)
-				(hide yes)
-			)
-		)
-		(property "Datasheet" ""
-			(at 43.18 162.56 0)
-			(effects
-				(font
-					(size 1.27 1.27)
-				)
-				(hide yes)
-			)
-		)
-		(property "Description" ""
-			(at 43.18 162.56 0)
-			(effects
-				(font
-					(size 1.27 1.27)
-				)
-				(hide yes)
-			)
-		)
-		(pin "1"
-		)
-		(instances
-			(project "WarpSE"
-				(path "/a5be2cb8-c68d-4180-8412-69a6b4c5b1d4/00000000-0000-0000-0000-00005f6da71d"
-					(reference "#PWR0153")
-					(unit 1)
-				)
-			)
-		)
-	)
-	(symbol
 		(lib_id "power:-5V")
 		(at 72.39 137.16 180)
@@
 	)
 	(symbol
-		(lib_id "Device:R_Small")
-		(at 43.18 160.02 0)
+		(lib_id "power:GND")
+		(at 33.02 162.56 0)
+		(mirror y)
 		(unit 1)
 		(exclude_from_sim no)
@@
 		(on_board yes)
 		(dnp no)
-		(property "Reference" "R27"
-			(at 44.45 158.75 0)
+		(property "Reference" "#PWR048"
+			(at 33.02 168.91 0)
 			(effects
 				(font
 					(size 1.27 1.27)
 				)
-				(justify left)
+				(hide yes)
 			)
 		)
-		(property "Value" "680"
-			(at 44.45 161.29 0)
+		(property "Value" "GND"
+			(at 33.02 166.37 0)
 			(effects
 				(font
 					(size 1.27 1.27)
 				)
-				(justify left)
 			)
 		)
-		(property "Footprint" "stdpads:R_0805"
-			(at 43.18 160.02 0)
+		(property "Footprint" ""
+			(at 33.02 162.56 0)
 			(effects
 				(font
@@
 			)
 		)
-		(property "Datasheet" "~"
-			(at 43.18 160.02 0)
+		(property "Datasheet" ""
+			(at 33.02 162.56 0)
 			(effects
 				(font
@@
 			)
 		)
-		(property "Description" "Resistor, small symbol"
-			(at 43.18 160.02 0)
+		(property "Description" ""
+			(at 33.02 162.56 0)
 			(effects
 				(font
@@
 		(pin "1"
 		)
-		(pin "2"
-		)
 		(instances
 			(project "WarpSE"
 				(path "/a5be2cb8-c68d-4180-8412-69a6b4c5b1d4/00000000-0000-0000-0000-00005f6da71d"
-					(reference "R27")
+					(reference "#PWR048")
 					(unit 1)
 				)
