File: RAM.kicad_sch (KiCad schematic)
At the start: 10 parts

Commit message: Switch to '030
Parts:
- added U?: SDRAM-16Mx16-TSOP2-54, stdpads:Winbond_TSOPII-54, symbol GW_RAM:SDRAM-16Mx16-TSOP2-54
Connections:
- net VSS is gone; now on net GND: U?.28 (VSS), U?.41 (VSS), U?.54 (VSS)
- net VSSQ is gone; now on net GND: U?.12 (VSSQ), U?.46 (VSSQ), U?.52 (VSSQ), U?.6 (VSSQ)
- net BA0: now also U?.20 (BA0)
- net BA1: now also U?.21 (BA1)
- net CKE: now also U?.37 (CKE)
- net GND: now also U?.12 (VSSQ), U?.28 (VSS), U?.41 (VSS), U?.46 (VSSQ), U?.52 (VSSQ), U?.54 (VSS), U?.6 (VSSQ)
- net RA0: now also U?.23 (A0)
- net RA1: now also U?.24 (A1)
- net RA10: now also U?.22 (A10)
- net RA11: now also U?.35 (A11)
- net RA2: now also U?.25 (A2)
- net RA3: now also U?.26 (A3)
- net RA4: now also U?.29 (A4)
- net RA5: now also U?.30 (A5)
- net RA6: now also U?.31 (A6)
- net RA7: now also U?.32 (A7)
- net RA8: now also U?.33 (A8)
- net RA9: now also U?.34 (A9)
- net VDD: now also U?.1 (VDD), U?.14 (VDD), U?.27 (VDD)
- net VDDQ: now also U?.3 (VDDQ), U?.43 (VDDQ), U?.49 (VDDQ), U?.9 (VDDQ)
- net ~{CAS}: now also U?.17 (~{CAS})
- net ~{RAS}: now also U?.18 (~{RAS})
- net ~{WE}: now also U?.16 (~{WE})
- net ~{CS}: now reaches U?.19 (~{CS})
- net ~{CS}: now also U?.19 (~{CS})
- net CLK renamed CLK0
- net DQMH renamed DQM0
- net DQML renamed DQM1
- new net CLK1: U?.38 (CLK)
- new net D16: U?.2 (DQ0)
- new net D17: U?.4 (DQ1)
- new net D18: U?.5 (DQ2)
- new net D19: U?.7 (DQ3)
- new net D20: U?.8 (DQ4)
- new net D21: U?.10 (DQ5)
- new net D22: U?.11 (DQ6)
- new net D23: U?.13 (DQ7)
- new net D24: U?.42 (DQ8)
- new net D25: U?.44 (DQ9)
- new net D26: U?.45 (DQ10)
- new net D27: U?.47 (DQ11)
- new net D28: U?.48 (DQ12)
- new net D29: U?.50 (DQ13)
- new net D30: U?.51 (DQ14)
- new net D31: U?.53 (DQ15)
- new net DQM2: U?.39 (DQMH)
- new net DQM3: U?.15 (DQML)
Other:
- moved on the sheet: C12, C13, C14, C15, C50, C51, U?

Commit message: more
Parts:
- removed U?: SDRAM-16Mx16-TSOP2-54, stdpads:Winbond_TSOPII-54, symbol GW_RAM:SDRAM-16Mx16-TSOP2-54
Connections:
- net ~{CS} is gone; now on net GND: U?.19 (~{CS})
- net A21: now reaches U?.36 (A12)
- net BA0 renamed A22
- net BA1 renamed A23
- net CLK0 renamed CLK
- net RA0 renamed A8
- net RA1 renamed A9
- net RA10 renamed A19
- net RA11 renamed A20
- net RA2 renamed A11
- net RA3 renamed A12
- net RA4 renamed A13
- net RA5 renamed A14
- net RA6 renamed A15
- net RA7 renamed A16
- net RA8 renamed A17
- net RA9 renamed A18

Commit message: more
Connections:
- net A8 is gone; now on net A9: U?.23 (A0)
- net A9: no longer U?.24 (A1)
- net DQM0 renamed DQMH
- net DQM1 renamed DQML
- new net A10: U?.24 (A1)
Changed lines of the file:
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@@
     (effects (font (size 1.27 1.27)) (justify left bottom))
   )
-  (label "A9" (at 90.17 88.9 180)
+  (label "A10" (at 90.17 88.9 180)
     (effects (font (size 1.27 1.27)) (justify right bottom))
   )
@@
     (effects (font (size 1.27 1.27)) (justify right bottom))
   )
-  (label "A8" (at 90.17 86.36 180)
+  (label "A9" (at 90.17 86.36 180)
     (effects (font (size 1.27 1.27)) (justify right bottom))
   )
@@
     (effects (font (size 1.27 1.27)) (justify right))
   )
-  (hierarchical_label "DQM0" (shape input) (at 115.57 121.92 0)
+  (hierarchical_label "DQMH" (shape input) (at 115.57 121.92 0)
     (effects (font (size 1.27 1.27)) (justify left))
   )
-  (hierarchical_label "DQM1" (shape input) (at 115.57 119.38 0)
+  (hierarchical_label "DQML" (shape input) (at 115.57 119.38 0)
     (effects (font (size 1.27 1.27)) (justify left))
   )

Commit message: more
Connections:
- net A10 renamed RA1
- net A11 renamed RA2
- net A12 renamed RA3
- net A13 renamed RA4
- net A14 renamed RA5
- net A15 renamed RA6
- net A16 renamed RA7
- net A17 renamed RA8
- net A18 renamed RA9
- net A19 renamed RA10
- net A20 renamed RA11
- net A21 renamed RA12
- net A22 renamed BA0
- net A23 renamed BA1
- net A9 renamed RA0
- net CKE renamed RCKE
- net CLK renamed RCLK
- net DQMH renamed RDQMH
- net DQML renamed RDQML
- net ~{CAS} renamed R~{CAS}
- net ~{RAS} renamed R~{RAS}
- net ~{WE} renamed R~{WE}

Commit message: idk
Parts:
- gave numbers to parts that had none: 1
Changed lines of the file:
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@@
   (symbol (lib_id "GW_RAM:SDRAM-16Mx16-TSOP2-54") (at 102.87 104.14 0) (unit 1)
     (in_bom yes) (on_board yes) (dnp no) (fields_autoplaced)
-    (property "Reference" "U?" (at 102.87 71.12 0)
+    (property "Reference" "U18" (at 102.87 71.12 0)
       (effects (font (size 1.27 1.27)))
     )
@@
       (project "WarpSE"
         (path "/a5be2cb8-c68d-4180-8412-69a6b4c5b1d4/00000000-0000-0000-0000-00005f723900"
-          (reference "U?") (unit 1)
+          (reference "U18") (unit 1)
         )
       )
@@
   (symbol (lib_id "power:GND") (at 118.11 125.73 0) (unit 1)
     (in_bom yes) (on_board yes) (dnp no)
-    (property "Reference" "#PWR?" (at 118.11 132.08 0)
+    (property "Reference" "#PWR0125" (at 118.11 132.08 0)
       (effects (font (size 1.27 1.27)) hide)
     )
@@
       (project "WarpSE"
         (path "/a5be2cb8-c68d-4180-8412-69a6b4c5b1d4/00000000-0000-0000-0000-00005f723900"
-          (reference "#PWR?") (unit 1)
+          (reference "#PWR0125") (unit 1)
         )
       )
@@
   (symbol (lib_id "power:GND") (at 90.17 137.16 0) (unit 1)
     (in_bom yes) (on_board yes) (dnp no)
-    (property "Reference" "#PWR?" (at 90.17 143.51 0)
+    (property "Reference" "#PWR0124" (at 90.17 143.51 0)
       (effects (font (size 1.27 1.27)) hide)
     )
@@
       (project "WarpSE"
         (path "/a5be2cb8-c68d-4180-8412-69a6b4c5b1d4/00000000-0000-0000-0000-00005f723900"
-          (reference "#PWR?") (unit 1)
+          (reference "#PWR0124") (unit 1)
         )
       )
