File: Prog.kicad_sch (KiCad schematic)
At the start: 31 parts, among them J2 JTAG, J3 microUSB, J4 microUSB, Q1 MMBT3904, Q2 MMBT3904, U12 CH340G, U19 24C08, U21 74LVC257APW, U7 74AHCT573PW, U9 CH341B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

Commit message: Update Prog.kicad_sch
Parts:
- added J5: USBROM, symbol Connector_Generic:Conn_02x05_Odd_Even
Connections:
- net B~{CS} is gone; now on net FF~{CS}: U21.4 (Za), U9.16 (~{CS}1)
- net F~{CS} is gone; now on net FR~{CS}: U21.7 (Zb), U9.15 (~{CS}0)
- net +3V3: now also J5.1 (Pin_1)
- net GND: now also J5.10 (Pin_10), J5.2 (Pin_2), J5.4 (Pin_4), J5.6 (Pin_6), J5.8 (Pin_8)
- net MOSI: now also U21.14 (D0)
- net SCK: now also U21.11 (C0)
- net WP: now also J5.3 (Pin_3)
- net SDA: now reaches R14.2, U19.5 (SDA), U9.23 (SDA)
- net SDA: now also J5.7 (Pin_7)
- net SCL: now reaches R13.2, U19.6 (SCL), U9.24 (SCL)
- net SCL: now also J5.5 (Pin_5)
- net FF~{CS}: now reaches U21.2 (A0)
- net FR~{CS}: now reaches U21.5 (B0)
- net USBRST: now reaches U9.2 (RSTI)
- net USBRST: now also J5.9 (Pin_9)
- net FPGA_B~{CS} renamed FPGA_FF~{CS}
- net FPGA_F~{CS} renamed FPGA_FR~{CS}
