File: RAMROM.kicad_sch (KiCad schematic)
At the start: 10 parts, among them U10 39SF040, U11 39SF040, U8 KM48C2100, U9 KM48C2100

Commit message: Documentation update
Connections:
- net A19 renamed B
Changed lines of the file:
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@@
-    (stroke (width 0) (type default) (color 0 0 0 0))
-  )
-  (bus_entry (at 205.74 119.38) (size -2.54 2.54)
     (stroke (width 0) (type default) (color 0 0 0 0))
   )
@@
     (stroke (width 0) (type default) (color 0 0 0 0))
   )
-  (bus_entry (at 205.74 71.12) (size -2.54 2.54)
-    (stroke (width 0) (type default) (color 0 0 0 0))
-  )
   (bus_entry (at 69.85 110.49) (size 2.54 -2.54)
     (stroke (width 0) (type default) (color 0 0 0 0))
@@
     (stroke (width 0) (type default) (color 0 0 0 0))
   )
-  (wire (pts (xy 210.82 119.38) (xy 205.74 119.38))
-    (stroke (width 0) (type default) (color 0 0 0 0))
-  )
   (bus (pts (xy 203.2 129.54) (xy 203.2 132.08))
     (stroke (width 0) (type default) (color 0 0 0 0))
@@
     (stroke (width 0) (type default) (color 0 0 0 0))
   )
-  (bus (pts (xy 203.2 121.92) (xy 203.2 124.46))
+  (bus (pts (xy 203.2 119.38) (xy 203.2 124.46))
     (stroke (width 0) (type default) (color 0 0 0 0))
   )
@@
     (stroke (width 0) (type default) (color 0 0 0 0))
   )
-  (bus (pts (xy 203.2 73.66) (xy 203.2 76.2))
-    (stroke (width 0) (type default) (color 0 0 0 0))
-  )
-  (bus (pts (xy 203.2 71.12) (xy 203.2 73.66))
+  (bus (pts (xy 203.2 71.12) (xy 203.2 76.2))
     (stroke (width 0) (type default) (color 0 0 0 0))
   )
@@
     (stroke (width 0) (type default) (color 0 0 0 0))
   )
-  (bus (pts (xy 203.2 119.38) (xy 203.2 121.92))
-    (stroke (width 0) (type default) (color 0 0 0 0))
-  )
   (wire (pts (xy 77.47 125.73) (xy 72.39 125.73))
     (stroke (width 0) (type default) (color 0 0 0 0))
@@
     (stroke (width 0) (type default) (color 0 0 0 0))
   )
-  (wire (pts (xy 210.82 71.12) (xy 205.74 71.12))
-    (stroke (width 0) (type default) (color 0 0 0 0))
-  )
   (bus (pts (xy 69.85 69.85) (xy 68.58 69.85))
     (stroke (width 0) (type default) (color 0 0 0 0))
@@
     (effects (font (size 1.27 1.27)) (justify right bottom))
   )
-  (label "A19" (at 210.82 119.38 180)
-    (effects (font (size 1.27 1.27)) (justify right bottom))
-  )
   (label "D14" (at 231.14 111.76 0)
     (effects (font (size 1.27 1.27)) (justify left bottom))
@@
   (label "D4" (at 231.14 50.8 0)
     (effects (font (size 1.27 1.27)) (justify left bottom))
-  )
-  (label "A19" (at 210.82 71.12 180)
-    (effects (font (size 1.27 1.27)) (justify right bottom))
   )
   (label "A11" (at 210.82 96.52 180)
@@
     (effects (font (size 1.27 1.27)) (justify left))
   )
+  (hierarchical_label "B" (shape input) (at 210.82 71.12 180)
+    (effects (font (size 1.27 1.27)) (justify right))
+  )
   (hierarchical_label "~{OE}" (shape input) (at 97.79 135.89 0)
     (effects (font (size 1.27 1.27)) (justify left))
@@
     (effects (font (size 1.27 1.27)) (justify left))
   )
+  (hierarchical_label "B" (shape input) (at 210.82 119.38 180)
+    (effects (font (size 1.27 1.27)) (justify right))
+  )
   (hierarchical_label "~{RAS}" (shape input) (at 97.79 92.71 0)

Commit message: idk
Parts:
- added C45: 10u, stdpads:C_0805, symbol Device:C_Small
Connections:
- net +5V: now also C45.1
- net GND: now also C45.2
Changed lines of the file:
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@@
   (junction (at 265.43 111.76) (diameter 0) (color 0 0 0 0)
   )
+  (junction (at 265.43 106.68) (diameter 0) (color 0 0 0 0)
+  )
   (junction (at 115.57 115.57) (diameter 0) (color 0 0 0 0)
   )
+  (junction (at 146.05 120.65) (diameter 0) (color 0 0 0 0)
+  )
   (junction (at 255.27 106.68) (diameter 0) (color 0 0 0 0)
   )
   (junction (at 125.73 115.57) (diameter 0) (color 0 0 0 0)
   )
-  (junction (at 146.05 120.65) (diameter 0) (color 0 0 0 0)
-  )
   (junction (at 135.89 120.65) (diameter 0) (color 0 0 0 0)
   )
+  (junction (at 275.59 111.76) (diameter 0) (color 0 0 0 0)
+  )
   (junction (at 125.73 120.65) (diameter 0) (color 0 0 0 0)
   )
@@
     (stroke (width 0) (type default) (color 0 0 0 0))
   )
+  (wire (pts (xy 265.43 106.68) (xy 275.59 106.68))
+    (stroke (width 0) (type default) (color 0 0 0 0))
+  )
   (wire (pts (xy 210.82 55.88) (xy 205.74 55.88))
     (stroke (width 0) (type default) (color 0 0 0 0))
@@
   )
   (wire (pts (xy 102.87 113.03) (xy 97.79 113.03))
+    (stroke (width 0) (type default) (color 0 0 0 0))
+  )
+  (wire (pts (xy 265.43 111.76) (xy 275.59 111.76))
     (stroke (width 0) (type default) (color 0 0 0 0))
   )
@@
     (pin "1")
     (pin "2")
-  )
-  (symbol (lib_id "power:GND") (at 146.05 120.65 0) (unit 1)
-    (in_bom yes) (on_board yes)
-    (property "Reference" "#PWR0135" (id 0) (at 146.05 127 0)
-      (effects (font (size 1.27 1.27)) hide)
-    )
-    (property "Value" "GND" (id 1) (at 146.05 124.46 0))
-    (property "Footprint" "" (id 2) (at 146.05 120.65 0)
-      (effects (font (size 1.27 1.27)) hide)
-    )
-    (property "Datasheet" "" (id 3) (at 146.05 120.65 0)
-      (effects (font (size 1.27 1.27)) hide)
-    )
-    (pin "1")
   )
   (symbol (lib_id "GW_RAM:Flash-512Kx8-PLCC-32") (at 220.98 58.42 0) (unit 1)
@@
     (pin "2")
   )
-  (symbol (lib_id "power:GND") (at 265.43 111.76 0) (unit 1)
-    (in_bom yes) (on_board yes)
-    (property "Reference" "#PWR0200" (id 0) (at 265.43 118.11 0)
-      (effects (font (size 1.27 1.27)) hide)
-    )
-    (property "Value" "GND" (id 1) (at 265.43 115.57 0))
-    (property "Footprint" "" (id 2) (at 265.43 111.76 0)
-      (effects (font (size 1.27 1.27)) hide)
-    )
-    (property "Datasheet" "" (id 3) (at 265.43 111.76 0)
-      (effects (font (size 1.27 1.27)) hide)
-    )
-    (pin "1")
-  )
   (symbol (lib_id "power:+5V") (at 97.79 67.31 0) (unit 1)
     (in_bom yes) (on_board yes)
@@
       (effects (font (size 1.27 1.27)) hide)
     )
+    (pin "1")
+  )
+  (symbol (lib_id "power:GND") (at 275.59 111.76 0) (unit 1)
+    (in_bom yes) (on_board yes)
+    (property "Reference" "#PWR0135" (id 0) (at 275.59 118.11 0)
+      (effects (font (size 1.27 1.27)) hide)
+    )
+    (property "Value" "GND" (id 1) (at 275.59 115.57 0))
+    (property "Footprint" "" (id 2) (at 275.59 111.76 0)
+      (effects (font (size 1.27 1.27)) hide)
+    )
+    (property "Datasheet" "" (id 3) (at 275.59 111.76 0)
+      (effects (font (size 1.27 1.27)) hide)
+    )
+    (pin "1")
+  )
+  (symbol (lib_id "Device:C_Small") (at 275.59 109.22 0) (unit 1)
+    (in_bom yes) (on_board yes)
+    (property "Reference" "C45" (id 0) (at 276.86 107.95 0)
+      (effects (font (size 1.27 1.27)) (justify left))
+    )
+    (property "Value" "10u" (id 1) (at 276.86 110.49 0)
+      (effects (font (size 1.27 1.27)) (justify left))
+    )
+    (property "Footprint" "stdpads:C_0805" (id 2) (at 275.59 109.22 0)
+      (effects (font (size 1.27 1.27)) hide)
+    )
+    (property "Datasheet" "~" (id 3) (at 275.59 109.22 0)
+      (effects (font (size 1.27 1.27)) hide)
+    )
+    (property "LCSC Part" "C15850" (id 4) (at 275.59 109.22 0)
+      (effects (font (size 1.27 1.27)) hide)
+    )
+    (pin "1")
+    (pin "2")
+  )
+  (symbol (lib_id "power:GND") (at 146.05 120.65 0) (unit 1)
+    (in_bom yes) (on_board yes)
+    (property "Reference" "#PWR0157" (id 0) (at 146.05 127 0)
+      (effects (font (size 1.27 1.27)) hide)
+    )
+    (property "Value" "GND" (id 1) (at 146.05 124.46 0))
+    (property "Footprint" "" (id 2) (at 146.05 120.65 0)
+      (effects (font (size 1.27 1.27)) hide)
+    )
+    (property "Datasheet" "" (id 3) (at 146.05 120.65 0)
+      (effects (font (size 1.27 1.27)) hide)
+    )

Commit message: Prototype
Parts:
- added C50, C51: 10u, stdpads:C_0805, symbol Device:C_Small
Connections:
- net A18 is gone; now on net RA8: U10.28 (A13), U11.26 (A9)
- net B is gone; now on net RA11: U10.29 (A14), U11.25 (A11)
- net +5V: now also C50.1, C51.1
- net GND: now also C50.2, C51.2
Changed lines of the file:
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@@
 (kicad_sch (version 20211123) (generator eeschema)
   (paper "A4")
+  (junction (at 156.21 115.57) (diameter 0) (color 0 0 0 0)
+  )
   (junction (at 265.43 111.76) (diameter 0) (color 0 0 0 0)
   )
+  (junction (at 166.37 120.65) (diameter 0) (color 0 0 0 0)
+  )
   (junction (at 265.43 106.68) (diameter 0) (color 0 0 0 0)
   )
@@
   (junction (at 125.73 115.57) (diameter 0) (color 0 0 0 0)
   )
+  (junction (at 156.21 120.65) (diameter 0) (color 0 0 0 0)
+  )
   (junction (at 135.89 120.65) (diameter 0) (color 0 0 0 0)
   )
+  (junction (at 146.05 115.57) (diameter 0) (color 0 0 0 0)
+  )
   (junction (at 275.59 111.76) (diameter 0) (color 0 0 0 0)
   )
@@
     (stroke (width 0) (type default) (color 0 0 0 0))
   )
-  (bus_entry (at 205.74 114.3) (size -2.54 2.54)
-    (stroke (width 0) (type default) (color 0 0 0 0))
-  )
   (bus_entry (at 69.85 118.11) (size 2.54 -2.54)
     (stroke (width 0) (type default) (color 0 0 0 0))
@@
     (stroke (width 0) (type default) (color 0 0 0 0))
   )
-  (bus_entry (at 205.74 68.58) (size -2.54 2.54)
-    (stroke (width 0) (type default) (color 0 0 0 0))
-  )
   (bus_entry (at 69.85 90.17) (size 2.54 -2.54)
     (stroke (width 0) (type default) (color 0 0 0 0))
@@
     (stroke (width 0) (type default) (color 0 0 0 0))
   )
-  (bus (pts (xy 203.2 114.3) (xy 203.2 116.84))
-    (stroke (width 0) (type default) (color 0 0 0 0))
-  )
   (bus (pts (xy 69.85 74.93) (xy 69.85 77.47))
     (stroke (width 0) (type default) (color 0 0 0 0))
@@
     (stroke (width 0) (type default) (color 0 0 0 0))
   )
-  (wire (pts (xy 210.82 114.3) (xy 205.74 114.3))
-    (stroke (width 0) (type default) (color 0 0 0 0))
-  )
   (wire (pts (xy 210.82 76.2) (xy 205.74 76.2))
     (stroke (width 0) (type default) (color 0 0 0 0))
@@
     (stroke (width 0) (type default) (color 0 0 0 0))
   )
+  (wire (pts (xy 146.05 120.65) (xy 156.21 120.65))
+    (stroke (width 0) (type default) (color 0 0 0 0))
+  )
   (wire (pts (xy 77.47 107.95) (xy 72.39 107.95))
     (stroke (width 0) (type default) (color 0 0 0 0))
@@
     (stroke (width 0) (type default) (color 0 0 0 0))
   )
+  (wire (pts (xy 146.05 115.57) (xy 156.21 115.57))
+    (stroke (width 0) (type default) (color 0 0 0 0))
+  )
   (wire (pts (xy 210.82 66.04) (xy 205.74 66.04))
     (stroke (width 0) (type default) (color 0 0 0 0))
@@
     (stroke (width 0) (type default) (color 0 0 0 0))
   )
-  (wire (pts (xy 210.82 68.58) (xy 205.74 68.58))
-    (stroke (width 0) (type default) (color 0 0 0 0))
-  )
   (wire (pts (xy 77.47 87.63) (xy 72.39 87.63))
     (stroke (width 0) (type default) (color 0 0 0 0))
@@
     (stroke (width 0) (type default) (color 0 0 0 0))
   )
-  (bus (pts (xy 203.2 71.12) (xy 203.2 76.2))
-    (stroke (width 0) (type default) (color 0 0 0 0))
-  )
   (bus (pts (xy 105.41 77.47) (xy 105.41 80.01))
     (stroke (width 0) (type default) (color 0 0 0 0))
@@
     (stroke (width 0) (type default) (color 0 0 0 0))
   )
+  (wire (pts (xy 156.21 115.57) (xy 166.37 115.57))
+    (stroke (width 0) (type default) (color 0 0 0 0))
+  )
   (bus (pts (xy 203.2 127) (xy 203.2 129.54))
     (stroke (width 0) (type default) (color 0 0 0 0))
@@
     (stroke (width 0) (type default) (color 0 0 0 0))
   )
-  (bus (pts (xy 203.2 68.58) (xy 203.2 71.12))
+  (bus (pts (xy 203.2 68.58) (xy 203.2 76.2))
     (stroke (width 0) (type default) (color 0 0 0 0))
   )
@@
     (stroke (width 0) (type default) (color 0 0 0 0))
   )
+  (wire (pts (xy 156.21 120.65) (xy 166.37 120.65))
+    (stroke (width 0) (type default) (color 0 0 0 0))
+  )
   (bus (pts (xy 203.2 96.52) (xy 203.2 99.06))
     (stroke (width 0) (type default) (color 0 0 0 0))
@@
     (stroke (width 0) (type default) (color 0 0 0 0))
   )
-  (bus (pts (xy 203.2 116.84) (xy 203.2 119.38))
+  (bus (pts (xy 203.2 114.3) (xy 203.2 119.38))
     (stroke (width 0) (type default) (color 0 0 0 0))
   )
@@
     (stroke (width 0) (type default) (color 0 0 0 0))
   )
+  (label "RA11" (at 210.82 71.12 180)
+    (effects (font (size 1.27 1.27)) (justify right bottom))
+  )
   (label "A6" (at 210.82 38.1 180)
     (effects (font (size 1.27 1.27)) (justify right bottom))
@@
     (effects (font (size 1.27 1.27)) (justify right bottom))
   )
-  (label "A18" (at 210.82 114.3 180)
-    (effects (font (size 1.27 1.27)) (justify right bottom))
-  )
   (label "D11" (at 231.14 104.14 0)
     (effects (font (size 1.27 1.27)) (justify left bottom))
@@
     (effects (font (size 1.27 1.27)) (justify right bottom))
   )
+  (label "RA8" (at 210.82 114.3 180)
+    (effects (font (size 1.27 1.27)) (justify right bottom))
+  )
   (label "D4" (at 97.79 85.09 0)
     (effects (font (size 1.27 1.27)) (justify left bottom))
   )
-  (label "A18" (at 210.82 68.58 180)
-    (effects (font (size 1.27 1.27)) (justify right bottom))
-  )
   (label "D6" (at 97.79 87.63 0)
     (effects (font (size 1.27 1.27)) (justify left bottom))
@@
   )
   (label "A9" (at 210.82 137.16 180)
+    (effects (font (size 1.27 1.27)) (justify right bottom))
+  )
+  (label "RA8" (at 210.82 68.58 180)
+    (effects (font (size 1.27 1.27)) (justify right bottom))
+  )
+  (label "RA11" (at 210.82 119.38 180)
     (effects (font (size 1.27 1.27)) (justify right bottom))
   )
@@
     (effects (font (size 1.27 1.27)) (justify left))
   )
-  (hierarchical_label "B" (shape input) (at 210.82 71.12 180)
-    (effects (font (size 1.27 1.27)) (justify right))
-  )
   (hierarchical_label "~{OE}" (shape input) (at 97.79 135.89 0)
     (effects (font (size 1.27 1.27)) (justify left))
@@
   (hierarchical_label "~{CAS}" (shape input) (at 97.79 90.17 0)
     (effects (font (size 1.27 1.27)) (justify left))
-  )
-  (hierarchical_label "B" (shape input) (at 210.82 119.38 180)
-    (effects (font (size 1.27 1.27)) (justify right))
   )
   (hierarchical_label "~{RAS}" (shape input) (at 97.79 92.71 0)
@@
     (pin "1")
   )
+  (symbol (lib_id "Device:C_Small") (at 166.37 118.11 0) (unit 1)
+    (in_bom yes) (on_board yes)
+    (property "Reference" "C51" (id 0) (at 167.64 116.84 0)
+      (effects (font (size 1.27 1.27)) (justify left))
+    )
+    (property "Value" "10u" (id 1) (at 167.64 119.38 0)
+      (effects (font (size 1.27 1.27)) (justify left))
+    )
+    (property "Footprint" "stdpads:C_0805" (id 2) (at 166.37 118.11 0)
+      (effects (font (size 1.27 1.27)) hide)
+    )
+    (property "Datasheet" "~" (id 3) (at 166.37 118.11 0)
+      (effects (font (size 1.27 1.27)) hide)
+    )
+    (property "LCSC Part" "C15850" (id 4) (at 166.37 118.11 0)
+      (effects (font (size 1.27 1.27)) hide)
+    )
+    (pin "1")
+    (pin "2")
+  )
+  (symbol (lib_id "Device:C_Small") (at 156.21 118.11 0) (unit 1)
+    (in_bom yes) (on_board yes)
+    (property "Reference" "C50" (id 0) (at 157.48 116.84 0)
+      (effects (font (size 1.27 1.27)) (justify left))
+    )
+    (property "Value" "10u" (id 1) (at 157.48 119.38 0)
+      (effects (font (size 1.27 1.27)) (justify left))
+    )
+    (property "Footprint" "stdpads:C_0805" (id 2) (at 156.21 118.11 0)
+      (effects (font (size 1.27 1.27)) hide)
+    )
+    (property "Datasheet" "~" (id 3) (at 156.21 118.11 0)
+      (effects (font (size 1.27 1.27)) hide)
+    )
+    (property "LCSC Part" "C15850" (id 4) (at 156.21 118.11 0)
+      (effects (font (size 1.27 1.27)) hide)
+    )
+    (pin "1")
+    (pin "2")
+  )
   (symbol (lib_id "power:GND") (at 275.59 111.76 0) (unit 1)
     (in_bom yes) (on_board yes)
@@
     (pin "2")
   )
-  (symbol (lib_id "power:GND") (at 146.05 120.65 0) (unit 1)
-    (in_bom yes) (on_board yes)
-    (property "Reference" "#PWR0157" (id 0) (at 146.05 127 0)
-      (effects (font (size 1.27 1.27)) hide)
-    )
-    (property "Value" "GND" (id 1) (at 146.05 124.46 0))
-    (property "Footprint" "" (id 2) (at 146.05 120.65 0)
-      (effects (font (size 1.27 1.27)) hide)
-    )
-    (property "Datasheet" "" (id 3) (at 146.05 120.65 0)
-      (effects (font (size 1.27 1.27)) hide)
-    )
+  (symbol (lib_id "power:GND") (at 166.37 120.65 0) (unit 1)
+    (in_bom yes) (on_board yes)
+    (property "Reference" "#PWR0132" (id 0) (at 166.37 127 0)
+      (effects (font (size 1.27 1.27)) hide)
+    )
+    (property "Value" "GND" (id 1) (at 166.37 124.46 0))
+    (property "Footprint" "" (id 2) (at 166.37 120.65 0)
+      (effects (font (size 1.27 1.27)) hide)
+    )
+    (property "Datasheet" "" (id 3) (at 166.37 120.65 0)
+      (effects (font (size 1.27 1.27)) hide)
+    )

Commit message: RC
Connections:
- net ROM~{CS} is gone; now on net GND: U10.22 (~{CS}), U11.22 (~{CS})
- net ~{OE}: no longer U10.24 (~{OE}), U11.24 (~{OE})
- new net ROM~{OE}: U10.24 (~{OE}), U11.24 (~{OE})
Other:
- company: (none) -> Garrett's Workshop
- title: (none) -> WarpSE (GW4410A)
Changed lines of the file:
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@@
 (kicad_sch (version 20230121) (generator eeschema)
   (paper "A4")
+  (title_block
+    (title "WarpSE (GW4410A)")
+    (date "2024-03-27")
+    (rev "1.0")
+    (company "Garrett's Workshop")
+  )
   (junction (at 156.21 115.57) (diameter 0) (color 0 0 0 0)
   )
@@
     (stroke (width 0) (type default))
   )
+  (wire (pts (xy 236.22 119.38) (xy 233.68 119.38))
+    (stroke (width 0) (type default))
+  )
   (bus (pts (xy 203.2 129.54) (xy 203.2 132.08))
     (stroke (width 0) (type default))
@@
     (stroke (width 0) (type default))
   )
+  (wire (pts (xy 233.68 63.5) (xy 233.68 68.58))
+    (stroke (width 0) (type default))
+  )
   (wire (pts (xy 210.82 76.2) (xy 205.74 76.2))
     (stroke (width 0) (type default))
@@
     (stroke (width 0) (type default))
   )
+  (wire (pts (xy 236.22 63.5) (xy 233.68 63.5))
+    (stroke (width 0) (type default))
+  )
   (wire (pts (xy 77.47 133.35) (xy 72.39 133.35))
     (stroke (width 0) (type default))
@@
     (stroke (width 0) (type default))
   )
+  (wire (pts (xy 233.68 119.38) (xy 233.68 124.46))
+    (stroke (width 0) (type default))
+  )
   (wire (pts (xy 231.14 55.88) (xy 238.76 55.88))
     (stroke (width 0) (type default))
@@
     (stroke (width 0) (type default))
   )
+  (wire (pts (xy 233.68 124.46) (xy 231.14 124.46))
+    (stroke (width 0) (type default))
+  )
   (bus (pts (xy 241.3 43.18) (xy 241.3 45.72))
     (stroke (width 0) (type default))
@@
     (stroke (width 0) (type default))
   )
+  (wire (pts (xy 233.68 68.58) (xy 231.14 68.58))
+    (stroke (width 0) (type default))
+  )
   (wire (pts (xy 97.79 80.01) (xy 102.87 80.01))
     (stroke (width 0) (type default))
@@
   (label "RA3" (at 77.47 133.35 180) (fields_autoplaced)
     (effects (font (size 1.27 1.27)) (justify right bottom))
-  )
-  (hierarchical_label "~{OE}" (shape input) (at 231.14 129.54 0) (fields_autoplaced)
-    (effects (font (size 1.27 1.27)) (justify left))
   )
   (hierarchical_label "D[15..0]" (shape bidirectional) (at 106.68 72.39 0) (fields_autoplaced)
@@
     (effects (font (size 1.27 1.27)) (justify left))
   )
-  (hierarchical_label "ROM~{CS}" (shape input) (at 231.14 124.46 0) (fields_autoplaced)
+  (hierarchical_label "ROM~{OE}" (shape input) (at 231.14 129.54 0) (fields_autoplaced)
     (effects (font (size 1.27 1.27)) (justify left))
   )
@@
     (effects (font (size 1.27 1.27)) (justify left))
   )
-  (hierarchical_label "~{OE}" (shape input) (at 231.14 73.66 0) (fields_autoplaced)
-    (effects (font (size 1.27 1.27)) (justify left))
-  )
   (hierarchical_label "L~{WE}" (shape input) (at 97.79 95.25 0) (fields_autoplaced)
     (effects (font (size 1.27 1.27)) (justify left))
@@
     (effects (font (size 1.27 1.27)) (justify left))
   )
-  (hierarchical_label "ROM~{CS}" (shape input) (at 231.14 68.58 0) (fields_autoplaced)
+  (hierarchical_label "ROM~{OE}" (shape input) (at 231.14 73.66 0) (fields_autoplaced)
     (effects (font (size 1.27 1.27)) (justify left))
   )
@@
     )
   )
+  (symbol (lib_id "power:GND") (at 236.22 119.38 0) (unit 1)
+    (in_bom yes) (on_board yes) (dnp no)
+    (property "Reference" "#PWR010" (at 236.22 125.73 0)
+      (effects (font (size 1.27 1.27)) hide)
+    )
+    (property "Value" "GND" (at 236.22 123.19 0)
+      (effects (font (size 1.27 1.27)))
+    )
+    (property "Footprint" "" (at 236.22 119.38 0)
+      (effects (font (size 1.27 1.27)) hide)
+    )
+    (property "Datasheet" "" (at 236.22 119.38 0)
+      (effects (font (size 1.27 1.27)) hide)
+    )
+    (pin "1")
+    (instances
+      (project "WarpSE"
+        (path "/a5be2cb8-c68d-4180-8412-69a6b4c5b1d4/00000000-0000-0000-0000-00005f723900"
+          (reference "#PWR010") (unit 1)
+        )
+      )
+    )
+  )
   (symbol (lib_id "Device:C_Small") (at 166.37 118.11 0) (unit 1)
     (in_bom yes) (on_board yes) (dnp no)
@@
         )
       )
+    )
+  )
+  (symbol (lib_id "power:GND") (at 236.22 63.5 0) (unit 1)
+    (in_bom yes) (on_board yes) (dnp no)
+    (property "Reference" "#PWR014" (at 236.22 69.85 0)
+      (effects (font (size 1.27 1.27)) hide)
+    )
+    (property "Value" "GND" (at 236.22 67.31 0)
+      (effects (font (size 1.27 1.27)))
+    )
+    (property "Footprint" "" (at 236.22 63.5 0)
+      (effects (font (size 1.27 1.27)) hide)
+    )
+    (property "Datasheet" "" (at 236.22 63.5 0)
+      (effects (font (size 1.27 1.27)) hide)
+    )
+    (pin "1")
+    (instances
+      (project "WarpSE"
+        (path "/a5be2cb8-c68d-4180-8412-69a6b4c5b1d4/00000000-0000-0000-0000-00005f723900"
+          (reference "#PWR014") (unit 1)
+        )
+      )
