File: RAMROM.kicad_sch (KiCad schematic)
At the start: 13 parts, among them U10 39SF040, U11 39SF040, U8 KM48C2100, U9 KM48C2100

Commit message: RC
Parts:
- U10, U11: LCSC Part C72257 -> C645935
Changed lines of the file:
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@@
   (title_block
     (title "WarpSE (GW4410A)")
-    (date "2024-03-27")
+    (date "2024-04-23")
     (rev "1.0")
     (company "Garrett's Workshop")
@@
       (effects (font (size 1.27 1.27)) hide)
     )
-    (property "Datasheet" "~" (at 125.73 118.11 0)
+    (property "Datasheet" "" (at 125.73 118.11 0)
       (effects (font (size 1.27 1.27)) hide)
     )
@@
       (effects (font (size 1.27 1.27)) hide)
     )
-    (property "Datasheet" "~" (at 115.57 118.11 0)
+    (property "Datasheet" "" (at 115.57 118.11 0)
       (effects (font (size 1.27 1.27)) hide)
     )
@@
       (effects (font (size 1.27 1.27)) hide)
     )
-    (property "Datasheet" "~" (at 135.89 118.11 0)
+    (property "Datasheet" "" (at 135.89 118.11 0)
       (effects (font (size 1.27 1.27)) hide)
     )
@@
       (effects (font (size 1.27 1.27)) hide)
     )
-    (property "Datasheet" "~" (at 146.05 118.11 0)
+    (property "Datasheet" "" (at 146.05 118.11 0)
       (effects (font (size 1.27 1.27)) hide)
     )
@@
       (effects (font (size 1.27 1.27)) hide)
     )
-    (property "Datasheet" "http://ww1.microchip.com/downloads/en/DeviceDoc/20005022C.pdf" (at 220.98 58.42 0)
-      (effects (font (size 1.27 1.27)) hide)
-    )
-    (property "LCSC Part" "C72257" (at 220.98 58.42 0)
+    (property "Datasheet" "" (at 220.98 58.42 0)
+      (effects (font (size 1.27 1.27)) hide)
+    )
+    (property "LCSC Part" "C645935" (at 220.98 58.42 0)
       (effects (font (size 1.27 1.27)) hide)
     )
@@
       (effects (font (size 1.27 1.27)) hide)
     )
-    (property "Datasheet" "http://ww1.microchip.com/downloads/en/DeviceDoc/20005022C.pdf" (at 220.98 114.3 0)
-      (effects (font (size 1.27 1.27)) hide)
-    )
-    (property "LCSC Part" "C72257" (at 220.98 114.3 0)
+    (property "Datasheet" "" (at 220.98 114.3 0)
+      (effects (font (size 1.27 1.27)) hide)
+    )
+    (property "LCSC Part" "C645935" (at 220.98 114.3 0)
       (effects (font (size 1.27 1.27)) hide)
     )
@@
       (effects (font (size 1.27 1.27)) hide)
     )
-    (property "Datasheet" "~" (at 265.43 109.22 0)
+    (property "Datasheet" "" (at 265.43 109.22 0)
       (effects (font (size 1.27 1.27)) hide)
     )
@@
       (effects (font (size 1.27 1.27)) hide)
     )
-    (property "Datasheet" "~" (at 255.27 109.22 0)
+    (property "Datasheet" "" (at 255.27 109.22 0)
       (effects (font (size 1.27 1.27)) hide)
     )
@@
       (effects (font (size 1.27 1.27)) hide)
     )
-    (property "Datasheet" "~" (at 166.37 118.11 0)
+    (property "Datasheet" "" (at 166.37 118.11 0)
       (effects (font (size 1.27 1.27)) hide)
     )
@@
       (effects (font (size 1.27 1.27)) hide)
     )
-    (property "Datasheet" "~" (at 156.21 118.11 0)
+    (property "Datasheet" "" (at 156.21 118.11 0)
       (effects (font (size 1.27 1.27)) hide)
     )
@@
       (effects (font (size 1.27 1.27)) hide)
     )
-    (property "Datasheet" "~" (at 275.59 109.22 0)
-      (effects (font (size 1.27 1.27)) hide)
-    )
+    (property "Datasheet" "" (at 275.59 109.22 0)
+      (effects (font (size 1.27 1.27)) hide)
+    )

Commit message: USB power
Parts:
- removed C45, C50, C51: 10u, stdpads:C_0805, symbol Device:C_Small
