File: Clk.kicad_sch (KiCad schematic)
At the start: 6 parts, among them U4 20M, U5 25M

Commit message: Toward final "A"
Parts:
- removed U4: 20M, stdpads:Crystal_SMD_3225-4Pin_3.2x2.5mm, symbol GW_Logic:Oscillator_4P
- added C53: 2u2, stdpads:C_0603, symbol Device:C_Small
- added R12, R3: 47, stdpads:R_0603, symbol Device:R_Small
- added U6, U7: 74LVC1G74DC, stdpads:NXP_VSSOP-8_2.3x2mm, symbol GW_Logic:741G74DC
- U5: value 25M -> 50M
Connections:
- net CK25EN is gone; now on net +3V3: U5.1 (EN)
- net +3V3: now also C53.1, U6.7 (~{S}), U6.8 (Vcc), U7.6 (~{R}), U7.7 (~{S}), U7.8 (Vcc)
- net GND: now also C53.2, U6.4 (GND), U7.4 (GND)
- net MCLK: now also R1.1, R12.2; no longer R1.2
- net RCLK: no longer names the net of R2.2
- net RCLK: now also R12.1, U7.5 (Q)
- new net: R1.2, U6.5 (Q)
- new net: R3.2, U5.3 (Output)
- new net: R3.1, U6.1 (CK), U7.1 (CK)
- new net: U7.2 (D), U7.3 (~{Q})
- new net: U6.2 (D), U6.3 (~{Q})
- new net FCLK: R2.1
- new net MCKE: U6.6 (~{R})
Other:
- moved on the sheet: R1, R2

Commit message: final version?
Parts:
- R12: value 47 -> DNP; LCSC Part C23182 -> (none)
Changed lines of the file:
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@@
       (effects (font (size 1.27 1.27)) (justify right))
     )
-    (property "Value" "47" (at 181.61 85.09 0)
+    (property "Value" "DNP" (at 181.61 85.09 0)
       (effects (font (size 1.27 1.27)) (justify right))
     )
@@
       (effects (font (size 1.27 1.27)) hide)
     )
-    (property "LCSC Part" "C23182" (at 180.34 83.82 0)
-      (effects (font (size 1.27 1.27)) hide)
-    )

Commit message: RC
Parts:
- added J5: CLKIN, stdpads:PinHeader_1x02_P2.54mm_Vertical, symbol Connector_Generic:Conn_01x02
- added J6: CLKDIS, stdpads:PinHeader_1x02_P2.54mm_Vertical, symbol Connector_Generic:Conn_01x02
- added R5: 47, stdpads:R_0603, symbol Device:R_Small
- added R8: 1k, stdpads:R_0603, symbol Device:R_Small
Connections:
- net +3V3: now also R8.2; no longer U5.1 (EN)
- net GND: now also J5.2 (Pin_2), J6.2 (Pin_2)
- net at R3.1, U6.1 (CK), U7.1 (CK): now also R5.1
- net at U7.2 (D), U7.3 (~{Q}): now also U6.2 (D)
- net at U6.3 (~{Q}): no longer U6.2 (D)
- new net: J6.1 (Pin_1), R8.1, U5.1 (EN)
- new net: J5.1 (Pin_1), R5.2
- no-connect marks 0 -> 1
Other:
- company: (none) -> Garrett's Workshop
- title: (none) -> WarpSE (GW4410A)
Changed lines of the file:
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@@
 (kicad_sch (version 20230121) (generator eeschema)
   (paper "A4")
+  (title_block
+    (title "WarpSE (GW4410A)")
+    (date "2024-03-27")
+    (rev "1.0")
+    (company "Garrett's Workshop")
+  )
+  (junction (at 138.43 77.47) (diameter 0) (color 0 0 0 0)
+  )
   (junction (at 88.9 105.41) (diameter 0) (color 0 0 0 0)
   )
@@
   (junction (at 184.15 72.39) (diameter 0) (color 0 0 0 0)
   )
+  (junction (at 148.59 92.71) (diameter 0) (color 0 0 0 0)
+  )
   (junction (at 143.51 77.47) (diameter 0) (color 0 0 0 0)
   )
+  (junction (at 113.03 77.47) (diameter 0) (color 0 0 0 0)
+  )
+  (junction (at 107.95 74.93) (diameter 0) (color 0 0 0 0)
+  )
   (junction (at 176.53 95.25) (diameter 0) (color 0 0 0 0)
   )
@@
   (junction (at 78.74 105.41) (diameter 0) (color 0 0 0 0)
   )
+  (no_connect (at 171.45 74.93))
   (wire (pts (xy 177.8 72.39) (xy 171.45 72.39))
     (stroke (width 0) (type default))
   )
-  (wire (pts (xy 148.59 92.71) (xy 148.59 107.95))
+  (wire (pts (xy 173.99 105.41) (xy 148.59 105.41))
     (stroke (width 0) (type default))
   )
@@
     (stroke (width 0) (type default))
   )
+  (wire (pts (xy 107.95 74.93) (xy 113.03 74.93))
+    (stroke (width 0) (type default))
+  )
+  (wire (pts (xy 173.99 97.79) (xy 173.99 105.41))
+    (stroke (width 0) (type default))
+  )
   (wire (pts (xy 180.34 87.63) (xy 180.34 86.36))
     (stroke (width 0) (type default))
@@
     (stroke (width 0) (type default))
   )
-  (wire (pts (xy 151.13 92.71) (xy 148.59 92.71))
-    (stroke (width 0) (type default))
-  )
   (wire (pts (xy 146.05 72.39) (xy 146.05 95.25))
     (stroke (width 0) (type default))
@@
     (stroke (width 0) (type default))
   )
-  (wire (pts (xy 148.59 107.95) (xy 173.99 107.95))
+  (wire (pts (xy 148.59 92.71) (xy 151.13 92.71))
     (stroke (width 0) (type default))
   )
@@
     (stroke (width 0) (type default))
   )
-  (wire (pts (xy 173.99 85.09) (xy 173.99 74.93))
+  (wire (pts (xy 138.43 77.47) (xy 143.51 77.47))
+    (stroke (width 0) (type default))
+  )
+  (wire (pts (xy 138.43 90.17) (xy 137.16 90.17))
     (stroke (width 0) (type default))
   )
@@
     (stroke (width 0) (type default))
   )
+  (wire (pts (xy 138.43 77.47) (xy 138.43 90.17))
+    (stroke (width 0) (type default))
+  )
+  (wire (pts (xy 105.41 77.47) (xy 113.03 77.47))
+    (stroke (width 0) (type default))
+  )
   (wire (pts (xy 182.88 72.39) (xy 184.15 72.39))
     (stroke (width 0) (type default))
@@
     (stroke (width 0) (type default))
   )
-  (wire (pts (xy 148.59 69.85) (xy 148.59 85.09))
+  (wire (pts (xy 148.59 105.41) (xy 148.59 92.71))
+    (stroke (width 0) (type default))
+  )
+  (wire (pts (xy 148.59 69.85) (xy 148.59 92.71))
     (stroke (width 0) (type default))
   )
@@
     (stroke (width 0) (type default))
   )
-  (wire (pts (xy 137.16 77.47) (xy 143.51 77.47))
-    (stroke (width 0) (type default))
-  )
-  (wire (pts (xy 173.99 107.95) (xy 173.99 97.79))
-    (stroke (width 0) (type default))
-  )
-  (wire (pts (xy 148.59 85.09) (xy 173.99 85.09))
-    (stroke (width 0) (type default))
-  )
-  (wire (pts (xy 173.99 74.93) (xy 171.45 74.93))
+  (wire (pts (xy 137.16 77.47) (xy 138.43 77.47))
+    (stroke (width 0) (type default))
+  )
+  (wire (pts (xy 105.41 74.93) (xy 107.95 74.93))
     (stroke (width 0) (type default))
   )
@@
     )
   )
+  (symbol (lib_id "power:+3V3") (at 107.95 69.85 0) (unit 1)
+    (in_bom yes) (on_board yes) (dnp no)
+    (property "Reference" "#PWR09" (at 107.95 73.66 0)
+      (effects (font (size 1.27 1.27)) hide)
+    )
+    (property "Value" "+3V3" (at 107.95 66.04 0)
+      (effects (font (size 1.27 1.27)))
+    )
+    (property "Footprint" "" (at 107.95 69.85 0)
+      (effects (font (size 1.27 1.27)) hide)
+    )
+    (property "Datasheet" "" (at 107.95 69.85 0)
+      (effects (font (size 1.27 1.27)) hide)
+    )
+    (pin "1")
+    (instances
+      (project "WarpSE"
+        (path "/a5be2cb8-c68d-4180-8412-69a6b4c5b1d4/00000000-0000-0000-0000-000061350d21"
+          (reference "#PWR09") (unit 1)
+        )
+      )
+    )
+  )
   (symbol (lib_id "Device:R_Small") (at 180.34 83.82 180) (unit 1)
     (in_bom yes) (on_board yes) (dnp no)
@@
     )
   )
+  (symbol (lib_id "power:GND") (at 132.08 92.71 0) (mirror y) (unit 1)
+    (in_bom yes) (on_board yes) (dnp no)
+    (property "Reference" "#PWR08" (at 132.08 99.06 0)
+      (effects (font (size 1.27 1.27)) hide)
+    )
+    (property "Value" "GND" (at 132.08 96.52 0)
+      (effects (font (size 1.27 1.27)))
+    )
+    (property "Footprint" "" (at 132.08 92.71 0)
+      (effects (font (size 1.27 1.27)) hide)
+    )
+    (property "Datasheet" "" (at 132.08 92.71 0)
+      (effects (font (size 1.27 1.27)) hide)
+    )
+    (pin "1")
+    (instances
+      (project "WarpSE"
+        (path "/a5be2cb8-c68d-4180-8412-69a6b4c5b1d4/00000000-0000-0000-0000-000061350d21"
+          (reference "#PWR08") (unit 1)
+        )
+      )
+    )
+  )
   (symbol (lib_id "power:GND") (at 171.45 100.33 0) (unit 1)
     (in_bom yes) (on_board yes) (dnp no)
@@
     )
   )
-  (symbol (lib_id "power:+3V3") (at 113.03 74.93 0) (mirror y) (unit 1)
-    (in_bom yes) (on_board yes) (dnp no)
-    (property "Reference" "#PWR014" (at 113.03 78.74 0)
-      (effects (font (size 1.27 1.27)) hide)
-    )
-    (property "Value" "+3V3" (at 113.03 71.12 0)
-      (effects (font (size 1.27 1.27)))
-    )
-    (property "Footprint" "" (at 113.03 74.93 0)
-      (effects (font (size 1.27 1.27)) hide)
-    )
-    (property "Datasheet" "" (at 113.03 74.93 0)
-      (effects (font (size 1.27 1.27)) hide)
-    )
-    (pin "1")
-    (instances
-      (project "WarpSE"
-        (path "/a5be2cb8-c68d-4180-8412-69a6b4c5b1d4/00000000-0000-0000-0000-000061350d21"
-          (reference "#PWR014") (unit 1)
-        )
-      )
-    )
-  )
   (symbol (lib_id "power:GND") (at 171.45 77.47 0) (unit 1)
     (in_bom yes) (on_board yes) (dnp no)
@@
     )
     (property "Value" "GND" (at 171.45 81.28 0)
-      (effects (font (size 1.27 1.27)))
+      (effects (font (size 1.27 1.27)) hide)
     )
     (property "Footprint" "" (at 171.45 77.47 0)
@@
     )
   )
+  (symbol (lib_id "Device:R_Small") (at 107.95 72.39 180) (unit 1)
+    (in_bom yes) (on_board yes) (dnp no)
+    (property "Reference" "R8" (at 109.22 71.12 0)
+      (effects (font (size 1.27 1.27)) (justify right))
+    )
+    (property "Value" "1k" (at 109.22 73.66 0)
+      (effects (font (size 1.27 1.27)) (justify right))
+    )
+    (property "Footprint" "stdpads:R_0603" (at 107.95 72.39 0)
+      (effects (font (size 1.27 1.27)) hide)
+    )
+    (property "Datasheet" "~" (at 107.95 72.39 0)
+      (effects (font (size 1.27 1.27)) hide)
+    )
+    (property "LCSC Part" "" (at 107.95 72.39 0)
+      (effects (font (size 1.27 1.27)) hide)
+    )
+    (pin "1")
+    (pin "2")
+    (instances
+      (project "WarpSE"
+        (path "/a5be2cb8-c68d-4180-8412-69a6b4c5b1d4/00000000-0000-0000-0000-000061350d21"
+          (reference "R8") (unit 1)
+        )
+      )
+    )
+  )
+  (symbol (lib_id "Connector_Generic:Conn_01x02") (at 100.33 74.93 0) (mirror y) (unit 1)
+    (in_bom yes) (on_board yes) (dnp no)
+    (property "Reference" "J6" (at 100.33 72.39 0)
+      (effects (font (size 1.27 1.27)))
+    )
+    (property "Value" "CLKDIS" (at 100.33 80.01 0)
+      (effects (font (size 1.27 1.27)))
+    )
+    (property "Footprint" "stdpads:PinHeader_1x02_P2.54mm_Vertical" (at 100.33 74.93 0)
+      (effects (font (size 1.27 1.27)) hide)
+    )
+    (property "Datasheet" "~" (at 100.33 74.93 0)
+      (effects (font (size 1.27 1.27)) hide)
+    )
+    (pin "1")
+    (pin "2")
+    (instances
+      (project "WarpSE"
+        (path "/a5be2cb8-c68d-4180-8412-69a6b4c5b1d4/00000000-0000-0000-0000-000061350d21"
+          (reference "J6") (unit 1)
+        )
+      )
+    )
+  )
+  (symbol (lib_id "Device:R_Small") (at 134.62 90.17 270) (unit 1)
+    (in_bom yes) (on_board yes) (dnp no)
+    (property "Reference" "R5" (at 134.62 86.36 90)
+      (effects (font (size 1.27 1.27)))
+    )
+    (property "Value" "47" (at 134.62 88.9 90)
+      (effects (font (size 1.27 1.27)) (justify bottom))
+    )
+    (property "Footprint" "stdpads:R_0603" (at 134.62 90.17 0)
+      (effects (font (size 1.27 1.27)) hide)
+    )
+    (property "Datasheet" "~" (at 134.62 90.17 0)
+      (effects (font (size 1.27 1.27)) hide)
+    )
+    (property "LCSC Part" "C23182" (at 134.62 90.17 0)
+      (effects (font (size 1.27 1.27)) hide)
+    )
+    (pin "1")
+    (pin "2")
+    (instances
+      (project "WarpSE"
+        (path "/a5be2cb8-c68d-4180-8412-69a6b4c5b1d4/00000000-0000-0000-0000-000061350d21"
+          (reference "R5") (unit 1)
+        )
+      )
+    )
+  )
   (symbol (lib_id "power:+3V3") (at 171.45 69.85 0) (unit 1)
     (in_bom yes) (on_board yes) (dnp no)
@@
         )
       )
+    )
+  )
+  (symbol (lib_id "Connector_Generic:Conn_01x02") (at 127 90.17 0) (mirror y) (unit 1)
+    (in_bom yes) (on_board yes) (dnp no)
+    (property "Reference" "J5" (at 127 87.63 0)
+      (effects (font (size 1.27 1.27)))
+    )
+    (property "Value" "CLKIN" (at 127 95.25 0)
+      (effects (font (size 1.27 1.27)))
+    )
+    (property "Footprint" "stdpads:PinHeader_1x02_P2.54mm_Vertical" (at 127 90.17 0)
+      (effects (font (size 1.27 1.27)) hide)
+    )
+    (property "Datasheet" "~" (at 127 90.17 0)
+      (effects (font (size 1.27 1.27)) hide)
+    )
+    (pin "1")
+    (pin "2")
+    (instances
+      (project "WarpSE"
+        (path "/a5be2cb8-c68d-4180-8412-69a6b4c5b1d4/00000000-0000-0000-0000-000061350d21"
+          (reference "J5") (unit 1)
+        )
+      )

Commit message: RC
Parts:
- added J7: PWR, stdpads:PinHeader_1x02_P2.54mm_Vertical, symbol Connector_Generic:Conn_01x02
- R8: LCSC Part (none) -> C21190
- U5: LCSC Part C32526 -> C717684
- U6, U7: LCSC Part (none) -> C503431
Connections:
- net GND: now also J7.2 (Pin_2)
- net CLKEN: now reaches J6.1 (Pin_1), R8.1, U5.1 (EN)
- new net +5V: J7.1 (Pin_1)
Other:
- moved on the sheet: J6, R8

Commit message: Before switching to SiT2001 oscillator
Parts:
- removed J5: CLKIN, stdpads:PinHeader_1x02_P2.54mm_Vertical, symbol Connector_Generic:Conn_01x02
- removed J6: CLKDIS, stdpads:PinHeader_1x02_P2.54mm_Vertical, symbol Connector_Generic:Conn_01x02
- removed J7: PWR, stdpads:PinHeader_1x02_P2.54mm_Vertical, symbol Connector_Generic:Conn_01x02
Connections:
- net CLKIN: now reaches R5.2

Commit message: Board changes
Parts:
- removed U5: 50M, stdpads:Crystal_SMD_3225-4Pin_3.2x2.5mm, symbol GW_Logic:Oscillator_4P
- added U5: SiT2001, stdpads:SOT-23-5, symbol GW_Logic:SiT2001
Connections:
- net +3V3: now also U5.4 (Vdd)
- net CLKEN: now also U5.3 (OE/~{ST})
- net GND: now also U5.1 (GND)
- net at R3.2: now also U5.5 (Output)
- no-connect marks 1 -> 2
Other:
- moved on the sheet: R8
