File: Buf.kicad_sch (KiCad schematic)
At the start: 32 parts, among them U13 74AHCT573PW, U15 74AHCT573PW, U16 74AHCT573PW, U17 74AHCT573PW, U18 74AHCT573PW, U19 74AHCT573PW, U2 74AHCT573PW, U20 74AHCT573PW, U21 74AHCT573PW, U22 74AHCT573PW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

Commit message: Final A?
Parts:
- removed R13, R22, R4, R9: 47, stdpads:R_0603, symbol Device:R_Small
Connections:
- net Aout20 is gone; now on net AccA20: R24.2, U2.5 (D3)
- net Aout21 is gone; now on net AccA21: R14.2, U2.4 (D2)
- net Aout23 is gone; now on net AccA23: R21.2, U2.2 (D0)
Other:
- moved on the sheet: U19, U20, U21, U22, U23, U24
