File: ClkBuf.kicad_sch (KiCad schematic)
At the start: 9 parts, among them U26 74LVC1G07GW, U27 74LVC1G07GW, U28 74LVC1G07GW

Commit message: final version?
Other:
- moved on the sheet: C26, C27, C28, R2, U28

Commit message: RC
Parts:
- removed C28: 2u2, stdpads:C_0603, symbol Device:C_Small
- added C21: 2u2, stdpads:C_0603, symbol Device:C_Small
- renumbered C26 to C48, C27 to C54, R2 to R17, R2 to R18, R2 to R7
Connections:
- net +3V3: now also C21.1
- net GND: now also C21.2
Other:
- company: (none) -> Garrett's Workshop
- title: (none) -> WarpSE (GW4410A)
Changed lines of the file:
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@@
 (kicad_sch (version 20230121) (generator eeschema)
   (paper "A4")
+  (title_block
+    (title "WarpSE (GW4410A)")
+    (date "2024-03-27")
+    (rev "1.0")
+    (company "Garrett's Workshop")
+  )
   (junction (at 113.03 133.35) (diameter 0) (color 0 0 0 0)
   )
@@
   (symbol (lib_id "Device:C_Small") (at 113.03 135.89 0) (unit 1)
     (in_bom yes) (on_board yes) (dnp no)
-    (property "Reference" "C26" (at 114.3 134.62 0)
+    (property "Reference" "C48" (at 114.3 134.62 0)
       (effects (font (size 1.27 1.27)) (justify left))
     )
@@
     (instances
       (project "WarpSE"
-        (path "/a5be2cb8-c68d-4180-8412-69a6b4c5b1d4/00000000-0000-0000-0000-00005f723173"
-          (reference "C26") (unit 1)
-        )
         (path "/a5be2cb8-c68d-4180-8412-69a6b4c5b1d4/fe631861-deed-4e97-a528-5baf968a7cc8"
           (reference "C48") (unit 1)
@@
   (symbol (lib_id "Device:R_Small") (at 146.05 88.9 270) (unit 1)
     (in_bom yes) (on_board yes) (dnp no)
-    (property "Reference" "R2" (at 146.05 85.09 90)
+    (property "Reference" "R18" (at 146.05 85.09 90)
       (effects (font (size 1.27 1.27)))
     )
@@
     (instances
       (project "WarpSE"
-        (path "/a5be2cb8-c68d-4180-8412-69a6b4c5b1d4/00000000-0000-0000-0000-000061350d21"
-          (reference "R2") (unit 1)
-        )
-        (path "/a5be2cb8-c68d-4180-8412-69a6b4c5b1d4/00000000-0000-0000-0000-000061aa52c4"
-          (reference "R20") (unit 1)
-        )
         (path "/a5be2cb8-c68d-4180-8412-69a6b4c5b1d4/fe631861-deed-4e97-a528-5baf968a7cc8"
           (reference "R18") (unit 1)
@@
     )
   )
+  (symbol (lib_id "power:GND") (at 133.35 138.43 0) (mirror y) (unit 1)
+    (in_bom yes) (on_board yes) (dnp no)
+    (property "Reference" "#PWR019" (at 133.35 144.78 0)
+      (effects (font (size 1.27 1.27)) hide)
+    )
+    (property "Value" "GND" (at 133.35 142.24 0)
+      (effects (font (size 1.27 1.27)))
+    )
+    (property "Footprint" "" (at 133.35 138.43 0)
+      (effects (font (size 1.27 1.27)) hide)
+    )
+    (property "Datasheet" "" (at 133.35 138.43 0)
+      (effects (font (size 1.27 1.27)) hide)
+    )
+    (pin "1")
+    (instances
+      (project "WarpSE"
+        (path "/a5be2cb8-c68d-4180-8412-69a6b4c5b1d4/fe631861-deed-4e97-a528-5baf968a7cc8"
+          (reference "#PWR019") (unit 1)
+        )
+      )
+    )
+  )
   (symbol (lib_id "Device:C_Small") (at 133.35 135.89 0) (unit 1)
     (in_bom yes) (on_board yes) (dnp no)
-    (property "Reference" "C28" (at 134.62 134.62 0)
+    (property "Reference" "C21" (at 134.62 134.62 0)
       (effects (font (size 1.27 1.27)) (justify left))
     )
@@
     (instances
       (project "WarpSE"
-        (path "/a5be2cb8-c68d-4180-8412-69a6b4c5b1d4/00000000-0000-0000-0000-00005f723173"
-          (reference "C28") (unit 1)
-        )
-        (path "/a5be2cb8-c68d-4180-8412-69a6b4c5b1d4/fe631861-deed-4e97-a528-5baf968a7cc8"
-          (reference "C55") (unit 1)
-        )
-      )
-    )
-  )
-  (symbol (lib_id "power:GND") (at 133.35 138.43 0) (mirror y) (unit 1)
-    (in_bom yes) (on_board yes) (dnp no)
-    (property "Reference" "#PWR0159" (at 133.35 144.78 0)
-      (effects (font (size 1.27 1.27)) hide)
-    )
-    (property "Value" "GND" (at 133.35 142.24 0)
-      (effects (font (size 1.27 1.27)))
-    )
-    (property "Footprint" "" (at 133.35 138.43 0)
-      (effects (font (size 1.27 1.27)) hide)
-    )
-    (property "Datasheet" "" (at 133.35 138.43 0)
-      (effects (font (size 1.27 1.27)) hide)
-    )
-    (pin "1")
-    (instances
-      (project "WarpSE"
-        (path "/a5be2cb8-c68d-4180-8412-69a6b4c5b1d4/00000000-0000-0000-0000-00005f723173"
-          (reference "#PWR0159") (unit 1)
-        )
-        (path "/a5be2cb8-c68d-4180-8412-69a6b4c5b1d4/fe631861-deed-4e97-a528-5baf968a7cc8"
-          (reference "#PWR019") (unit 1)
+        (path "/a5be2cb8-c68d-4180-8412-69a6b4c5b1d4/fe631861-deed-4e97-a528-5baf968a7cc8"
+          (reference "C21") (unit 1)
         )
       )
@@
   (symbol (lib_id "Device:R_Small") (at 146.05 104.14 270) (unit 1)
     (in_bom yes) (on_board yes) (dnp no)
-    (property "Reference" "R2" (at 146.05 100.33 90)
+    (property "Reference" "R17" (at 146.05 100.33 90)
       (effects (font (size 1.27 1.27)))
     )
@@
     (instances
       (project "WarpSE"
-        (path "/a5be2cb8-c68d-4180-8412-69a6b4c5b1d4/00000000-0000-0000-0000-000061350d21"
-          (reference "R2") (unit 1)
-        )
-        (path "/a5be2cb8-c68d-4180-8412-69a6b4c5b1d4/00000000-0000-0000-0000-000061aa52c4"
-          (reference "R20") (unit 1)
-        )
         (path "/a5be2cb8-c68d-4180-8412-69a6b4c5b1d4/fe631861-deed-4e97-a528-5baf968a7cc8"
           (reference "R17") (unit 1)
@@
   (symbol (lib_id "Device:C_Small") (at 123.19 135.89 0) (unit 1)
     (in_bom yes) (on_board yes) (dnp no)
-    (property "Reference" "C27" (at 124.46 134.62 0)
+    (property "Reference" "C54" (at 124.46 134.62 0)
       (effects (font (size 1.27 1.27)) (justify left))
     )
@@
     (instances
       (project "WarpSE"
-        (path "/a5be2cb8-c68d-4180-8412-69a6b4c5b1d4/00000000-0000-0000-0000-00005f723173"
-          (reference "C27") (unit 1)
-        )
         (path "/a5be2cb8-c68d-4180-8412-69a6b4c5b1d4/fe631861-deed-4e97-a528-5baf968a7cc8"
           (reference "C54") (unit 1)
@@
   (symbol (lib_id "power:+3V3") (at 113.03 133.35 0) (unit 1)
     (in_bom yes) (on_board yes) (dnp no)
-    (property "Reference" "#PWR0158" (at 113.03 137.16 0)
+    (property "Reference" "#PWR018" (at 113.03 137.16 0)
       (effects (font (size 1.27 1.27)) hide)
     )
@@
     (instances
       (project "WarpSE"
-        (path "/a5be2cb8-c68d-4180-8412-69a6b4c5b1d4/00000000-0000-0000-0000-00005f723173"
-          (reference "#PWR0158") (unit 1)
-        )
         (path "/a5be2cb8-c68d-4180-8412-69a6b4c5b1d4/fe631861-deed-4e97-a528-5baf968a7cc8"
           (reference "#PWR018") (unit 1)
@@
   (symbol (lib_id "Device:R_Small") (at 146.05 119.38 270) (unit 1)
     (in_bom yes) (on_board yes) (dnp no)
-    (property "Reference" "R2" (at 146.05 115.57 90)
+    (property "Reference" "R7" (at 146.05 115.57 90)
       (effects (font (size 1.27 1.27)))
     )
@@
     (instances
       (project "WarpSE"
-        (path "/a5be2cb8-c68d-4180-8412-69a6b4c5b1d4/00000000-0000-0000-0000-000061350d21"
-          (reference "R2") (unit 1)
-        )
-        (path "/a5be2cb8-c68d-4180-8412-69a6b4c5b1d4/00000000-0000-0000-0000-000061aa52c4"
-          (reference "R20") (unit 1)
-        )
         (path "/a5be2cb8-c68d-4180-8412-69a6b4c5b1d4/fe631861-deed-4e97-a528-5baf968a7cc8"
           (reference "R7") (unit 1)

Commit message: RC
Parts:
- U26, U27, U28: value 74LVC1G07GW -> 74LVC1G34GW; symbol GW_Logic:741G04GW -> GW_Logic:741G32GW; LCSC Part (none) -> C455045
Connections:
- net GND: now also U26.1 (A), U27.1 (A), U28.1 (A)
- no-connect marks 3 -> 0
Changed lines of the file:
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@@
   (title_block
     (title "WarpSE (GW4410A)")
-    (date "2024-03-27")
+    (date "2024-04-23")
     (rev "1.0")
     (company "Garrett's Workshop")
@@
   (junction (at 133.35 138.43) (diameter 0) (color 0 0 0 0)
   )
+  (junction (at 121.92 104.14) (diameter 0) (color 0 0 0 0)
+  )
   (junction (at 123.19 133.35) (diameter 0) (color 0 0 0 0)
   )
+  (junction (at 121.92 88.9) (diameter 0) (color 0 0 0 0)
+  )
   (junction (at 123.19 138.43) (diameter 0) (color 0 0 0 0)
   )
-  (no_connect (at 123.19 114.3))
-  (no_connect (at 123.19 83.82))
-  (no_connect (at 123.19 99.06))
+  (wire (pts (xy 119.38 80.01) (xy 121.92 80.01))
+    (stroke (width 0) (type default))
+  )
   (wire (pts (xy 123.19 133.35) (xy 133.35 133.35))
     (stroke (width 0) (type default))
   )
+  (wire (pts (xy 121.92 80.01) (xy 121.92 83.82))
+    (stroke (width 0) (type default))
+  )
   (wire (pts (xy 143.51 119.38) (xy 142.24 119.38))
     (stroke (width 0) (type default))
@@
     (stroke (width 0) (type default))
   )
+  (wire (pts (xy 121.92 104.14) (xy 121.92 114.3))
+    (stroke (width 0) (type default))
+  )
+  (wire (pts (xy 119.38 88.9) (xy 121.92 88.9))
+    (stroke (width 0) (type default))
+  )
+  (wire (pts (xy 121.92 88.9) (xy 121.92 99.06))
+    (stroke (width 0) (type default))
+  )
   (wire (pts (xy 149.86 119.38) (xy 148.59 119.38))
+    (stroke (width 0) (type default))
+  )
+  (wire (pts (xy 119.38 104.14) (xy 121.92 104.14))
     (stroke (width 0) (type default))
   )
@@
       (effects (font (size 1.27 1.27)) hide)
     )
-    (property "Datasheet" "~" (at 113.03 135.89 0)
+    (property "Datasheet" "" (at 113.03 135.89 0)
       (effects (font (size 1.27 1.27)) hide)
     )
@@
     )
   )
-  (symbol (lib_id "GW_Logic:741G04GW") (at 132.08 101.6 0) (unit 1)
+  (symbol (lib_id "GW_Logic:741G32GW") (at 132.08 101.6 0) (unit 1)
     (in_bom yes) (on_board yes) (dnp no)
     (property "Reference" "U27" (at 132.08 95.25 0)
       (effects (font (size 1.27 1.27)))
     )
-    (property "Value" "74LVC1G07GW" (at 132.08 107.95 0)
+    (property "Value" "74LVC1G34GW" (at 132.08 107.95 0)
       (effects (font (size 1.27 1.27)))
     )
@@
     (property "Datasheet" "" (at 132.08 106.68 0)
       (effects (font (size 1.524 1.524)) hide)
+    )
+    (property "LCSC Part" "C455045" (at 132.08 101.6 0)
+      (effects (font (size 1.27 1.27)) hide)
     )
     (pin "1")
@@
       (effects (font (size 1.27 1.27)) hide)
     )
-    (property "Datasheet" "~" (at 146.05 88.9 0)
+    (property "Datasheet" "" (at 146.05 88.9 0)
       (effects (font (size 1.27 1.27)) hide)
     )
@@
         (path "/a5be2cb8-c68d-4180-8412-69a6b4c5b1d4/fe631861-deed-4e97-a528-5baf968a7cc8"
           (reference "#PWR02") (unit 1)
-        )
-      )
-    )
-  )
-  (symbol (lib_id "power:GND") (at 121.92 88.9 0) (unit 1)
-    (in_bom yes) (on_board yes) (dnp no)
-    (property "Reference" "#PWR06" (at 121.92 95.25 0)
-      (effects (font (size 1.27 1.27)) hide)
-    )
-    (property "Value" "GND" (at 121.92 92.71 0)
-      (effects (font (size 1.27 1.27)))
-    )
-    (property "Footprint" "" (at 121.92 88.9 0)
-      (effects (font (size 1.27 1.27)) hide)
-    )
-    (property "Datasheet" "" (at 121.92 88.9 0)
-      (effects (font (size 1.27 1.27)) hide)
-    )
-    (pin "1")
-    (instances
-      (project "WarpSE"
-        (path "/a5be2cb8-c68d-4180-8412-69a6b4c5b1d4/fe631861-deed-4e97-a528-5baf968a7cc8"
-          (reference "#PWR06") (unit 1)
         )
       )
@@
       (effects (font (size 1.27 1.27)) hide)
     )
-    (property "Datasheet" "~" (at 133.35 135.89 0)
+    (property "Datasheet" "" (at 133.35 135.89 0)
       (effects (font (size 1.27 1.27)) hide)
     )
@@
       (effects (font (size 1.27 1.27)) hide)
     )
-    (property "Datasheet" "~" (at 146.05 104.14 0)
+    (property "Datasheet" "" (at 146.05 104.14 0)
       (effects (font (size 1.27 1.27)) hide)
     )
@@
         (path "/a5be2cb8-c68d-4180-8412-69a6b4c5b1d4/fe631861-deed-4e97-a528-5baf968a7cc8"
           (reference "R17") (unit 1)
+        )
+      )
+    )
+  )
+  (symbol (lib_id "power:GND") (at 119.38 88.9 0) (unit 1)
+    (in_bom yes) (on_board yes) (dnp no)
+    (property "Reference" "#PWR06" (at 119.38 95.25 0)
+      (effects (font (size 1.27 1.27)) hide)
+    )
+    (property "Value" "GND" (at 119.38 92.71 0)
+      (effects (font (size 1.27 1.27)))
+    )
+    (property "Footprint" "" (at 119.38 88.9 0)
+      (effects (font (size 1.27 1.27)) hide)
+    )
+    (property "Datasheet" "" (at 119.38 88.9 0)
+      (effects (font (size 1.27 1.27)) hide)
+    )
+    (pin "1")
+    (instances
+      (project "WarpSE"
+        (path "/a5be2cb8-c68d-4180-8412-69a6b4c5b1d4/fe631861-deed-4e97-a528-5baf968a7cc8"
+          (reference "#PWR06") (unit 1)
         )
       )
@@
       (effects (font (size 1.27 1.27)) hide)
     )
-    (property "Datasheet" "~" (at 123.19 135.89 0)
+    (property "Datasheet" "" (at 123.19 135.89 0)
       (effects (font (size 1.27 1.27)) hide)
     )
@@
     )
   )
-  (symbol (lib_id "GW_Logic:741G04GW") (at 132.08 86.36 0) (unit 1)
+  (symbol (lib_id "GW_Logic:741G32GW") (at 132.08 86.36 0) (unit 1)
     (in_bom yes) (on_board yes) (dnp no)
     (property "Reference" "U26" (at 132.08 80.01 0)
       (effects (font (size 1.27 1.27)))
     )
-    (property "Value" "74LVC1G07GW" (at 132.08 92.71 0)
+    (property "Value" "74LVC1G34GW" (at 132.08 92.71 0)
       (effects (font (size 1.27 1.27)))
     )
@@
     (property "Datasheet" "" (at 132.08 91.44 0)
       (effects (font (size 1.524 1.524)) hide)
+    )
+    (property "LCSC Part" "C455045" (at 132.08 86.36 0)
+      (effects (font (size 1.27 1.27)) hide)
     )
     (pin "1")
@@
     )
   )
-  (symbol (lib_id "GW_Logic:741G04GW") (at 132.08 116.84 0) (unit 1)
+  (symbol (lib_id "GW_Logic:741G32GW") (at 132.08 116.84 0) (unit 1)
     (in_bom yes) (on_board yes) (dnp no)
     (property "Reference" "U28" (at 132.08 110.49 0)
       (effects (font (size 1.27 1.27)))
     )
-    (property "Value" "74LVC1G07GW" (at 132.08 123.19 0)
+    (property "Value" "74LVC1G34GW" (at 132.08 123.19 0)
       (effects (font (size 1.27 1.27)))
     )
@@
     (property "Datasheet" "" (at 132.08 121.92 0)
       (effects (font (size 1.524 1.524)) hide)
+    )
+    (property "LCSC Part" "C455045" (at 132.08 116.84 0)
+      (effects (font (size 1.27 1.27)) hide)
     )
     (pin "1")
@@
     )
   )
-  (symbol (lib_id "power:GND") (at 121.92 104.14 0) (unit 1)
-    (in_bom yes) (on_board yes) (dnp no)
-    (property "Reference" "#PWR04" (at 121.92 110.49 0)
-      (effects (font (size 1.27 1.27)) hide)
-    )
-    (property "Value" "GND" (at 121.92 107.95 0)
-      (effects (font (size 1.27 1.27)))
-    )
-    (property "Footprint" "" (at 121.92 104.14 0)
-      (effects (font (size 1.27 1.27)) hide)
-    )
-    (property "Datasheet" "" (at 121.92 104.14 0)
+  (symbol (lib_id "power:GND") (at 119.38 80.01 0) (unit 1)
+    (in_bom yes) (on_board yes) (dnp no)
+    (property "Reference" "#PWR028" (at 119.38 86.36 0)
+      (effects (font (size 1.27 1.27)) hide)
+    )
+    (property "Value" "GND" (at 119.38 83.82 0)
+      (effects (font (size 1.27 1.27)))
+    )
+    (property "Footprint" "" (at 119.38 80.01 0)
+      (effects (font (size 1.27 1.27)) hide)
+    )
+    (property "Datasheet" "" (at 119.38 80.01 0)
+      (effects (font (size 1.27 1.27)) hide)
+    )
+    (pin "1")
+    (instances
+      (project "WarpSE"
+        (path "/a5be2cb8-c68d-4180-8412-69a6b4c5b1d4/fe631861-deed-4e97-a528-5baf968a7cc8"
+          (reference "#PWR028") (unit 1)
+        )
+      )
+    )
+  )
+  (symbol (lib_id "power:GND") (at 119.38 104.14 0) (unit 1)
+    (in_bom yes) (on_board yes) (dnp no)
+    (property "Reference" "#PWR04" (at 119.38 110.49 0)
+      (effects (font (size 1.27 1.27)) hide)
+    )
+    (property "Value" "GND" (at 119.38 107.95 0)
+      (effects (font (size 1.27 1.27)))
+    )
+    (property "Footprint" "" (at 119.38 104.14 0)
+      (effects (font (size 1.27 1.27)) hide)
+    )
+    (property "Datasheet" "" (at 119.38 104.14 0)
       (effects (font (size 1.27 1.27)) hide)
     )
@@
       (effects (font (size 1.27 1.27)) hide)
     )
-    (property "Datasheet" "~" (at 146.05 119.38 0)
-      (effects (font (size 1.27 1.27)) hide)
-    )
+    (property "Datasheet" "" (at 146.05 119.38 0)
+      (effects (font (size 1.27 1.27)) hide)
+    )

Commit message: Board prerelease revision 3 with USB power, A[23:20] remapping
Parts:
- added R29: 22k, stdpads:R_0805, symbol Device:R_Small
Connections:
- net C8M: now also R29.2
- new net +5Vin: R29.1
Changed lines of the file:
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@@
+	)
+	(junction
+		(at 114.3 101.6)
+		(diameter 0)
+		(color 0 0 0 0)
 	)
 	(junction
@@
 	(wire
 		(pts
+			(xy 114.3 93.98) (xy 113.03 93.98)
+		)
+		(stroke
+			(width 0)
+			(type default)
+		)
+	)
+	(wire
+		(pts
 			(xy 119.38 80.01) (xy 121.92 80.01)
 		)
@@
 	(wire
 		(pts
+			(xy 114.3 100.33) (xy 114.3 101.6)
+		)
+		(stroke
+			(width 0)
+			(type default)
+		)
+	)
+	(wire
+		(pts
+			(xy 114.3 101.6) (xy 121.92 101.6)
+		)
+		(stroke
+			(width 0)
+			(type default)
+		)
+	)
+	(wire
+		(pts
+			(xy 114.3 93.98) (xy 114.3 95.25)
+		)
+		(stroke
+			(width 0)
+			(type default)
+		)
+	)
+	(wire
+		(pts
 			(xy 119.38 104.14) (xy 121.92 104.14)
 		)
@@
 			(width 0)
 			(type default)
+		)
+	)
+	(wire
+		(pts
+			(xy 113.03 101.6) (xy 114.3 101.6)
+		)
+		(stroke
+			(width 0)
+			(type default)
+		)
+	)
+	(global_label "+5Vin"
+		(shape input)
+		(at 113.03 93.98 180)
+		(fields_autoplaced yes)
+		(effects
+			(font
+				(size 1.27 1.27)
+			)
+			(justify right)
+		)
+		(property "Intersheetrefs" "${INTERSHEET_REFS}"
+			(at 105.0747 93.98 0)
+			(effects
+				(font
+					(size 1.27 1.27)
+				)
+				(justify right)
+				(hide yes)
+			)
 		)
 	)
@@
 	(hierarchical_label "C8M"
 		(shape input)
-		(at 121.92 101.6 180)
+		(at 113.03 101.6 180)
 		(fields_autoplaced yes)
 		(effects
@@
 					(unit 1)
 				)
+			)
+		)
+	)
+	(symbol
+		(lib_id "Device:R_Small")
+		(at 114.3 97.79 0)
+		(unit 1)
+		(exclude_from_sim no)
+		(in_bom yes)
+		(on_board yes)
+		(dnp no)
+		(property "Reference" "R29"
+			(at 115.57 96.52 0)
+			(effects
+				(font
+					(size 1.27 1.27)
+				)
+				(justify left)
+			)
+		)
+		(property "Value" "22k"
+			(at 115.57 99.06 0)
+			(effects
+				(font
+					(size 1.27 1.27)
+				)
+				(justify left)
+			)
+		)
+		(property "Footprint" "stdpads:R_0805"
+			(at 114.3 97.79 0)
+			(effects
+				(font
+					(size 1.27 1.27)
+				)
+				(hide yes)
+			)
+		)
+		(property "Datasheet" "~"
+			(at 114.3 97.79 0)
+			(effects
+				(font
+					(size 1.27 1.27)
+				)
+				(hide yes)
+			)
+		)
+		(property "Description" "Resistor, small symbol"
+			(at 114.3 97.79 0)
+			(effects
+				(font
+					(size 1.27 1.27)
+				)
+				(hide yes)
+			)
+		)
+		(pin "1"
+		)
+		(pin "2"
+		)
+		(instances
+			(project "WarpSE"
+				(path "/a5be2cb8-c68d-4180-8412-69a6b4c5b1d4/fe631861-deed-4e97-a528-5baf968a7cc8"
+					(reference "R29")
+					(unit 1)
+				)

Commit message: Before remove first clock input buffer
Parts:
- R29: LCSC Part (none) -> C17560
- U26, U27, U28: value 74LVC1G34GW -> 74LVC1G32GW; LCSC Part C455045 -> C12516
Changed lines of the file:
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@@
 			)
 		)
-		(property "Value" "74LVC1G34GW"
+		(property "Value" "74LVC1G32GW"
 			(at 132.08 107.95 0)
 			(effects
@@
 			)
 		)
-		(property "LCSC Part" "C455045"
+		(property "LCSC Part" "C12516"
 			(at 132.08 101.6 0)
 			(effects
@@
 			)
 		)
-		(property "Value" "74LVC1G34GW"
+		(property "Value" "74LVC1G32GW"
 			(at 132.08 92.71 0)
 			(effects
@@
 			)
 		)
-		(property "LCSC Part" "C455045"
+		(property "LCSC Part" "C12516"
 			(at 132.08 86.36 0)
 			(effects
@@
 			)
 		)
-		(property "Value" "74LVC1G34GW"
+		(property "Value" "74LVC1G32GW"
 			(at 132.08 123.19 0)
 			(effects
@@
 			)
 		)
-		(property "LCSC Part" "C455045"
+		(property "LCSC Part" "C12516"
 			(at 132.08 116.84 0)
 			(effects
@@
 			(at 114.3 97.79 0)
 			(effects
+				(font
+					(size 1.27 1.27)
+				)
+				(hide yes)
+			)
+		)
+		(property "LCSC Part" "C17560"
+			(at 114.3 97.79 0)
+			(effects
