File: MC68k.kicad_sch (KiCad schematic)
At the start: 3 parts, among them U14 MC68HC000FN20

Commit message: Prototype
Changed lines of the file:
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@@
       (effects (font (size 1.27 1.27)) hide)
     )
-    (property "Value" "+5V" (id 1) (at 30.48 49.53 0))
+    (property "Value" "+5V" (id 1) (at 33.02 50.8 0))
     (property "Footprint" "" (id 2) (at 30.48 53.34 0)
       (effects (font (size 1.27 1.27)) hide)

Commit message: RC
Other:
- company: (none) -> Garrett's Workshop
- title: (none) -> WarpSE (GW4410A)
Changed lines of the file:
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@@
 (kicad_sch (version 20230121) (generator eeschema)
   (paper "A4")
+  (title_block
+    (title "WarpSE (GW4410A)")
+    (date "2024-03-27")
+    (rev "1.0")
+    (company "Garrett's Workshop")
+  )
   (junction (at 43.18 187.96) (diameter 0) (color 0 0 0 0)
   )
