File: WarpSE.kicad_sch (KiCad schematic)
At the start: 9 parts

Commit message: Final A?
Other:
- sheet Clk.sch ports: added CLKEN, CLKIN; removed none
- sheet Control ports: added CLKEN, CLKIN; removed none

Commit message: just a schematic change?
Connections:
- no-connect marks 0 -> 1
Other:
- sheet Control ports: added none; removed Mac~{BG}
Changed lines of the file:
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@@
 		(color 0 0 0 0)
 	)
+	(no_connect
+		(at 38.1 127)
+	)
 	(bus
 		(pts
@@
 		(pts
 			(xy 71.12 59.69) (xy 111.76 59.69)
-		)
-		(stroke
-			(width 0)
-			(type default)
-		)
-	)
-	(wire
-		(pts
-			(xy 38.1 127) (xy 81.28 127)
 		)
 		(stroke
@@
 			(effects
 				(font
-					(size 1.27 1.27)
-				)
-				(justify left)
-			)
-		)
-		(pin "Mac~{BG}" input
-			(at 81.28 127 180)
-			(effects
-				(font
