File: PowerAdapter/SEPowerAdapter.kicad_pcb (KiCad board)
At the start: 2 copper layers, 48 x 94.6 mm, 38 parts, among them J1 XOR, J2 ATX, J3 Mac, J4 VGA, U1 LM7905_TO220, U2 74LVC86AD, U3 74LVC86AD

Commit message: idk
Parts:
- added C17: 1n, stdpads:C_0805, F.Cu at (100.2, 177.9)
- added C18: 10u, stdpads:C_0805, F.Cu at (92.3, 164.0)
- added C19: 10u, stdpads:C_0805, F.Cu at (74.8, 188.8)
- added C20: 10u, stdpads:C_0805, F.Cu at (74.8, 185.3)
- added C22: 10u, stdpads:C_0805, F.Cu at (74.8, 181.6)
- added C23: 10u, stdpads:C_0805, F.Cu at (74.8, 177.3)
- added J3: SE, stdpads:Molex_Mini-Fit_Jr_5569-14A1_2x07_P4.20mm_Horizontal, F.Cu at (65.8, 127.5)
- added R12: 47, stdpads:R_0805, F.Cu at (102.0, 180.0)
- added R13: 2k2, stdpads:R_0805, F.Cu at (111.3, 189.6)
- added R14: 22k, stdpads:R_0805, F.Cu at (92.3, 161.8)
- J4: renamed from J3; value Mac -> Classic
- R1, R2, R3: value 1k -> 2k2
- moved R2 93.1 mm to (35.1, 132.7)
- moved J1 82.7 mm to (39.2, 128.3), turned to 0 degrees
- moved R3 82.5 mm to (35.1, 130.6), turned to 180 degrees
- moved R1 79.5 mm to (35.1, 128.6), turned to 180 degrees
- moved C15 48.4 mm to (74.8, 117.8)
- moved C1 48.4 mm to (74.8, 114.0)
- moved C12 48.4 mm to (74.8, 110.5)
- moved C6 48.4 mm to (74.8, 122.4)
- moved J4 19.1 mm to (65.8, 171.9)
- moved REF** 19.0 mm to (61.3, 100.8)
- moved REF** 19.0 mm to (64.4, 191.1)
- moved C16 1.78 mm to (106.3, 189.6)
- moved R5 1.59 mm to (113.3, 181.2)
- moved U2 1.59 mm to (107.9, 183.8)
- moved R4 1.59 mm to (113.3, 185.0)
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- renumbered J4 to J5
Connections:
- J1 pad 1: /HSx -> /VSx
- J1 pad 3: /VSx -> /HSx
- J4 pad 1: GND -> +12V
- J4 pad 10: /HSi -> GND
- J4 pad 11: /VSi -> GND
- J4 pad 12: +5V -> GND
- J4 pad 13: +5V -> GND
- J4 pad 14: +12V -> GND
- J4 pad 2: GND -> +5V
- J4 pad 3: GND -> +5V
- J4 pad 4: GND -> /VSi
- J4 pad 5: GND -> /HSi
- J4 pad 6: -5V -> /Ci
- J4 pad 7: -12V -> /AUDIO
- J4 pad 8: GND -> -12V
- J4 pad 9: /Ci -> /PBL
- R2 pad 1: /VSx -> /HSx
- R3 pad 1: /HSx -> /VSx
- U2 pad 1: /HSi -> /HSf
- U2 pad 10: GND -> /HSx
- U2 pad 2: /HSx -> GND
- U2 pad 8: unconnected-(U2-Pad8) -> Net-(R12-Pad1)
- U2 pad 9: GND -> /HSi
Routing:
- net /VSi: track 24.2 -> 108.5 mm, vias 0 -> 2
- net +3V3: track 158.7 -> 83.4 mm
- net /HSi: track 24.1 -> 92.3 mm, vias 0 -> 2
- net /Ci: track 42.5 -> 109.1 mm, vias 2 -> 0
- net /Cx: track 63.5 -> 10.5 mm, vias 2 -> 0
- net /VSx: track 32.2 -> 6.80 mm
- net -5V: track 43.9 -> 19.2 mm
- net /HSx: track 28.2 -> 7.06 mm
- net /HSf: track 0.00 -> 20.6 mm, vias 0 -> 2
- net -12V: track 85.8 -> 102.6 mm
- net +5V: track 128.8 -> 142.8 mm, vias 0 -> 1
- net +12V: track 45.6 -> 39.4 mm
- net GND: track 94.0 -> 97.8 mm, vias 86 -> 70
- net Net-(R12-Pad1): track 0.00 -> 2.41 mm
- net Net-(C17-Pad1): track 0.00 -> 2.03 mm
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- added copper zone on In2.Cu, net +3V3
- added copper zone on In1.Cu, net GND
Other:
- board size 48 x 94.6 mm -> 67.1 x 94.6 mm
- copper layers 2 -> 4
- board text added: "Classic"
- board text added: "SE"

Commit message: Fixing this up some more
Parts:
- moved R2 76.7 mm to (88.5, 187.6)
- moved R3 76.7 mm to (88.5, 185.6)
- moved J1 76.7 mm to (92.6, 183.3)
- moved R1 76.7 mm to (88.5, 183.5)
Routing:
- net +12V: track 39.4 -> 70.7 mm, vias 0 -> 1
- net +5V: track 142.8 -> 114.0 mm, vias 1 -> 2
- net -12V: track 102.6 -> 125.5 mm, vias 0 -> 1

Commit message: Toward final "A"
Parts:
- added REF**: XKB_TS-1187A, stdpads:XKB_TS-1187A, F.Cu at (88.4, 188.5)
- moved J1 6.70 mm to (89.7, 177.2)
- moved R1 6.70 mm to (85.6, 177.5)
- moved R2 6.70 mm to (85.6, 181.6)
- moved R3 6.70 mm to (85.6, 179.6)
Routing:
- net /HSi: track 92.3 -> 95.7 mm
- net /Ci: track 109.1 -> 112.1 mm
- net /VSi: track 108.5 -> 111.3 mm
