File: PowerAdapter/SEPowerAdapter.kicad_sch (KiCad schematic)
At the start: 6 parts

Commit message: More work on power adapter
Parts:
- added C1, C10, C11, C12, C13, C14, C15, C16, C2, C3, C4, C5, C6, C7, C8, C9: 2u2, stdpads:C_0805, symbol Device:C_Small
- added J1: XOR, Connector_PinHeader_2.54mm:PinHeader_2x03_P2.54mm_Vertical, symbol Connector_Generic:Conn_02x03_Odd_Even
- added J3: Mac, Connector_Molex:Molex_Mini-Fit_Jr_5569-14A1_2x07_P4.20mm_Horizontal, symbol Connector_Generic:Conn_02x07_Top_Bottom
- added J4: VGA, Connector_Dsub:DSUB-15-HD_Female_Horizontal_P2.29x1.98mm_EdgePinOffset3.03mm_Housed_MountingHolesOffset4.94mm, symbol Connector:DB15_Female_HighDensity_MountingHoles
- added R1, R2, R3: 1k, stdpads:R_0805, symbol Device:R_Small
- added R10, R6, R8: 150, stdpads:R_0805, symbol Device:R_Small
- added R11, R7, R9: 130, stdpads:R_0805, symbol Device:R_Small
- added R4, R5: 47, stdpads:R_0805, symbol Device:R_Small
- added U1: LM7905_TO220, Package_TO_SOT_THT:TO-220-3_Horizontal_TabDown, symbol Regulator_Linear:LM7905_TO220
- added unit 4 of U2
- added unit 5 of U2
- added unit 3 of U2
- added unit 5 of U3
- added unit 4 of U3
- J2: renamed from J?; value Conn_02x12_Top_Bottom -> ATX; footprint (none) -> Connector_Molex:Molex_Mini-Fit_Jr_5569-24A1_2x12_P4.20mm_Horizontal
- U2, U3: renamed from U?; footprint (none) -> stdpads:SOIC-14_3.9mm
Connections:
- net Bo: now also J4.3, R10.2, R11.2; no longer U3.3
- net Ci: now also U3.4, U3.9, J3.9 (Pin_9); no longer U3.1, U3.1
- net Cx: now also U3.10, U3.5, J1.5 (Pin_5), R1.1; no longer U3.2, U3.2
- net Go: now also J4.2, R8.2, R9.2; no longer U3.3
- net HSi: now also J3.10 (Pin_10)
- net HSo: now also J4.13, R4.2; no longer U2.3
- net HSx: now also J1.1 (Pin_1), R3.1
- net Ro: now also J4.1, R6.2, R7.2; no longer U3.3
- net VSi: now also U2.4, J3.11 (Pin_11); no longer U2.1
- net VSo: now also J4.14, R5.2; no longer U2.3
- net VSx: now also U2.5, J1.3 (Pin_3), R2.1; no longer U2.2
- net +3V3: now reaches J2.1 (Pin_1)
- net +3V3: now also J2.12 (Pin_12), J2.13 (Pin_13), J2.2 (Pin_2), C10.1, C16.1, C8.1, C9.1, R1.2, R2.2, R3.2, U2.14 (VCC), U3.14 (VCC)
- net +12V: now reaches J2.10 (Pin_10)
- net +12V: now also J2.11 (Pin_11), C1.1, C2.1, J3.14 (Pin_14)
- net -12V: now reaches J2.14 (Pin_14)
- net -12V: now also C11.2, C12.2, C13.2, J3.7 (Pin_7), U1.2 (VI)
- net GND: now reaches J2.15 (Pin_15)
- net GND: now also J2.17 (Pin_17), J2.18 (Pin_18), J2.19 (Pin_19), J2.24 (Pin_24), J2.3 (Pin_3), J2.5 (Pin_5), J2.7 (Pin_7), C1.2, C10.2, C11.1, C12.1, C13.1, C14.1, C15.1, C16.2, C2.2, C3.2, C4.2, C5.2, C6.2, C7.2, C8.2, C9.2, J1.2 (Pin_2), J1.4 (Pin_4), J1.6 (Pin_6), J3.1 (Pin_1), J3.2 (Pin_2), J3.3 (Pin_3), J3.4 (Pin_4), J3.5 (Pin_5), J3.8 (Pin_8), J4.0, J4.10, J4.5, J4.6, J4.7, J4.8, R11.1, R7.1, R9.1, U1.1 (GND), U2.10, U2.12, U2.13, U2.7 (GND), U2.9, U3.12, U3.13, U3.7 (GND)
- net ~{PS_ON}: now reaches J2.16 (Pin_16)
- net +5V: now reaches J2.21 (Pin_21)
- net +5V: now also J2.22 (Pin_22), J2.23 (Pin_23), J2.4 (Pin_4), J2.6 (Pin_6), C3.1, C4.1, C5.1, C6.1, C7.1, J3.12 (Pin_12), J3.13 (Pin_13)
- net PWR_OK: now reaches J2.8 (Pin_8)
- net +5VP: now reaches J2.9 (Pin_9)
- new net: R5.1, U2.6
- new net: R10.1, U3.8
- new net: R8.1, U3.6
- new net: R6.1, U3.3
- new net: R4.1, U2.3
- new net -5V: C14.2, C15.2, J3.6 (Pin_6), U1.3 (VO)
- no-connect marks 0 -> 9
Other:
- moved on the sheet: U2A, U2B, U3A, U3B, U3C

Commit message: Finished power adapter?
Parts:
- C1, C10, C11, C12, C13, C14, C15, C16, C2, C3, C4, C5, C6, C7, C8, C9: value 2u2 -> 10u; LCSC Part (none) -> C15850
- J1: LCSC Part (none) -> C65114
- J2: LCSC Part (none) -> C477841
- J3: footprint Connector_Molex:Molex_Mini-Fit_Jr_5569-14A1_2x07_P4.20mm_Horizontal -> stdpads:Molex_Mini-Fit_Jr_5569-14A1_2x07_P4.20mm_Horizontal; LCSC Part (none) -> C52216
- J4: LCSC Part (none) -> C75754
- R1, R2, R3: LCSC Part (none) -> C17513
- R10, R6, R8: LCSC Part (none) -> C17471
- R11, R7, R9: LCSC Part (none) -> C17437
- R4, R5: LCSC Part (none) -> C17714
- U1: footprint Package_TO_SOT_THT:TO-220-3_Horizontal_TabDown -> stdpads:TO-220-3_Horizontal_TabDown; LCSC Part (none) -> C9411
- U2, U3: LCSC Part (none) -> C548853
Connections:
- net at U3.8: now also R6.1; no longer R10.1
- net at U3.3: now also R10.1; no longer R6.1
Other:
- moved on the sheet: U3A, U3C

Commit message: idk
Parts:
- added C17: 1n, stdpads:C_0805, symbol Device:C_Small
- added C18, C19, C20, C22, C23: 10u, stdpads:C_0805, symbol Device:C_Small
- added D1: 1N4148, symbol Device:D_Small_Filled
- added J4: Classic, stdpads:Molex_Mini-Fit_Jr_5569-14A1_2x07_P4.20mm_Horizontal, symbol Connector_Generic:Conn_02x07_Top_Bottom
- added R12: 47, stdpads:R_0805, symbol Device:R_Small
- added R13: 2k2, stdpads:R_0805, symbol Device:R_Small
- added R14: 22k, stdpads:R_0805, symbol Device:R_Small
- added U4: 74HCT74D, symbol 74xx:74LS74
- J3: value Mac -> SE
- R1, R2, R3: value 1k -> 2k2
- renumbered J4 to J5
Connections:
- net +12V: now also C19.1, J4.1 (Pin_1)
- net +5V: now also C22.1, C23.1, J4.2 (Pin_2), J4.3 (Pin_3), R13.1
- net +5VP: now also D1.1 (K), R14.1, U4.2 (D)
- net -12V: now also C20.2, J4.8 (Pin_8)
- net Ci: now also J4.6 (Pin_6)
- net GND: now also U2.2, C18.2, C19.2, C20.1, C22.2, C23.2, J4.10 (Pin_10), J4.11 (Pin_11), J4.12 (Pin_12), J4.13 (Pin_13), J4.14 (Pin_14); no longer U2.10, U2.9
- net HSi: now also U2.9, J4.5 (Pin_5); no longer U2.1
- net HSx: now also J1.3 (Pin_3), R2.1, U2.10; no longer J1.1 (Pin_1), R3.1, U2.2
- net VSi: now also J4.4 (Pin_4)
- net VSx: now also J1.1 (Pin_1), R3.1; no longer J1.3 (Pin_3), R2.1
- net ~{PS_ON}: now also U4.6 (~{Q})
- net at U2.8: now also R12.1
- new net: C17.1, R12.2
- new net AUDIO: J4.7 (Pin_7)
- new net HSf: C17.2, R13.2, U2.1
- new net PBL: J4.9 (Pin_9)
- new net ~{BTN_OFF}: U4.4 (~{S})
- new net ~{BTN_ON}: U4.3 (C)
- new net ~{POR}: C18.1, D1.2 (A), R14.2, U4.1 (~{R})
Other:
- moved on the sheet: C1, C10, C11, C12, C13, C14, C15, C16, C2, C3, C4, C5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

Commit message: Toward final "A"
Parts:
- removed unit 1 of U2
- added C21, C24: 10u, stdpads:C_0805, symbol Device:C_Small
- added D2: Schottky, stdpads:D_SOD-123, symbol Device:D_Schottky_Small_Filled
- added R15: 1k, stdpads:R_0805, symbol Device:R_Small
- added R16, R17: 10k, stdpads:R_0805, symbol Device:R_Small
- added U5, U6: 74LVC1G14GW, stdpads:SOT-353, symbol GW_Logic:741G04GW
- added U7: 741G74DC, stdpads:NXP_VSSOP-8_2.3x2mm, symbol GW_Logic:741G74DC
- R13: value 2k2 -> 200
Connections:
- net +3V3: now also R16.1, R17.2, U5.5 (Vcc), U6.5 (Vcc), U7.6 (~{R}), U7.8 (Vcc)
- net +5V: no longer R13.1
- net GND: now also R13.2, C21.2, C24.2, U5.3 (GND), U6.3 (GND), U7.4 (GND)
- net HSf: now also R13.1, U5.2 (A); no longer R13.2
- net ~{PS_ON}: now also D2.2 (A)
- net at R4.1: now also U5.4 (Y)
- new net: C24.1, R15.2, R17.1, U6.2 (A)
- new net: U6.4 (Y), U7.1 (CK)
- new net: U7.2 (D), U7.3 (~{Q})
- new net: D2.1 (K), U7.5 (Q)
- new net: C21.1, R16.2, U7.7 (~{S})
Other:
- moved on the sheet: C17, J2, J3, J4, R10, R11, R12, R13, R4, R5, R6, R7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
